File: laboratorio/projetos/kicad/dd_cmos/DD_CMOS.sch (KiCad schematic (older format))
At the start: 33 parts

Commit message: Algumas revisões nos circuitos.
Parts:
- removed AFF? (x2): 7 SEGMENT DISPLAY, symbol 7SEGMENTS
- added AFF? (x2): HDSP-7xxx-C, symbol HDSP-7xxx-C
- Q?: value 2N1711 -> BC547
Connections:
- wire segments 147 -> 128
Other:
- note added: "+"
- note added: "-"
- note added: "Dado Digital usando CMOS"
- moved on the sheet: R?

Commit message: Ajustes de leiaute.
Parts:
- added P?: CONN_01X02, ck, symbol CONN_01X02
- added P? (x2): CONN_01X02, symbol CONN_01X02
- D1: renamed from D?; value D -> 1N4148
- gave numbers to parts that had none: 29
- renumbered . to .14
Connections:
- net labels removed: +12C, Lamp
- wire segments 128 -> 131
Other:
- note removed: "+"
- note removed: "-"
- note removed: "CLOCK"
- moved on the sheet: AFF1, AFF2, R1

Commit message: Atualizações no esquemático do Dado Digital CMOS.
Parts:
- removed K1: RELAY, symbol RELAY_2RT
- removed P?: CONN_01X02, ck, symbol CONN_01X02
- removed P?: CONN_01X02, symbol CONN_01X02
- removed U1: 74LS132, symbol 74LS132
- added P1, P2, P3: CONN_01X02, ~, symbol CONN_01X02
- added RL1: FINDER-40.51, symbol FINDER-40.51
- added U1: 4093, symbol 4093
- C1: value C -> 1uF
- C2: value C -> 10uF
- R1: value 1k -> 10k
- gave numbers to parts that had none: 1
- renumbered AFF2 to AFF1, AFF1 to AFF2
Connections:
- net labels added: +12V, GNDA, VSS, ck
- wire segments 131 -> 147
- no-connect marks 0 -> 5
Other:
- note added: "+12V"
- note added: "+5V"
- note added: "clock"
- note added: "dezena"
- note added: "lâmpada\n 12V"
- note added: "unidade"
- note removed: "Dado Digital usando CMOS"
- moved on the sheet: AFF1, AFF2, P4, R1, U6

Commit message: Pequenos ajustes e definição de licença.
Changed lines of the file:
@@
 Comp "Escola de Engenharia Mauá - IMT"
 Comment1 "ETE102 - Fundamentos de Circuitos Digitais"
-Comment2 "Gabarito"
-Comment3 ""
+Comment2 "Licença: CC-BY-SA (http://creativecommons.org/licenses/by-sa/4.0/)"
+Comment3 "GABARITO"
 Comment4 ""
 $EndDescr
@@
 	5000 3400 5150 3400
 Wire Wire Line
-	5000 2200 5100 2200
+	5050 2200 5100 2200
 Wire Wire Line
 	2200 1950 2200 2200
@@
 	1150 2850 1100 2850
 Wire Wire Line
-	1150 2750 1150 2850
-Wire Wire Line
 	1150 2950 1150 3000
-Text Label 1150 2750 0    60   ~ 0
-ck
-Text Label 5000 2200 2    60   ~ 0
-ck
 $Comp
 L VSS #PWR021
@@
 Text Notes 10950 5150 1    60   ~ 0
 lâmpada\n  12V
+Text GLabel 1150 2850 2    60   Input ~ 0
+ck
+Text GLabel 5050 2200 0    60   Input ~ 0
+ck
 $EndSCHEMATC

Commit message: Ajuste de lógica para parar/disparar contagem. Definições de "power flag".
Connections:
- net at U2.1 (Q): no longer U3.1 (CK)
- net at U2.2 (~Q), U4.6 (Ia=b): now also U3.1 (CK)
- no-connect marks 5 -> 6
Changed lines of the file:
@@
 	2200 3650 2200 3550
 Wire Wire Line
-	4600 2100 5100 2100
+	4750 2100 5100 2100
 Wire Wire Line
 	5000 3400 5000 2700
 Wire Wire Line
-	4600 4050 4600 3300
-Wire Wire Line
-	4600 3300 4600 2100
-Wire Wire Line
-	5150 3300 4600 3300
-Connection ~ 4600 3300
+	4750 4050 4750 3300
+Wire Wire Line
+	4750 3300 4750 2100
+Wire Wire Line
+	5150 3300 4750 3300
+Connection ~ 4750 3300
 Wire Wire Line
 	3850 1600 3850 1650
@@
 	3600 1600 3600 1750
 Wire Wire Line
-	4450 5150 7500 5150
-Wire Wire Line
-	4450 5150 4450 2400
+	4650 5150 7500 5150
 Wire Wire Line
 	10800 1650 10700 1650
@@
 	2950 4050 3850 4050
 Wire Wire Line
-	3850 4050 4600 4050
+	3850 4050 4750 4050
 Wire Wire Line
 	7350 2200 7500 2200
@@
 $EndComp
 Wire Wire Line
-	1150 1550 1100 1550
+	1100 1550 1150 1550
+Wire Wire Line
+	1150 1550 1350 1550
 Wire Wire Line
 	1150 1550 1150 1500
@@
 	1100 2300 1150 2300
 Wire Wire Line
-	1150 2200 1100 2200
+	1150 2300 1350 2300
+Wire Wire Line
+	1100 2200 1150 2200
+Wire Wire Line
+	1150 2200 1350 2200
 Wire Wire Line
 	1150 2150 1150 2200
@@
 	2300 2300 2350 2300
 Connection ~ 2300 2200
-Wire Wire Line
-	4450 2000 5100 2000
 Wire Wire Line
 	1350 1650 1350 1700
@@
 Text GLabel 5050 2200 0    60   Input ~ 0
 ck
+Wire Wire Line
+	4450 2400 4650 2400
+Wire Wire Line
+	4650 2000 4650 2400
+Wire Wire Line
+	4650 2400 4650 5150
+Wire Wire Line
+	5100 2000 4650 2000
+Connection ~ 4650 2400
+NoConn ~ 4450 2000
+$Comp
+L PWR_FLAG #FLG027
+U 1 1 5757DD02
+P 1350 2350
+F 0 "#FLG027" H 1350 2445 50  0001 C CNN
+F 1 "PWR_FLAG" H 1350 2530 50  0001 C CNN
+F 2 "" H 1350 2350 50  0000 C CNN
+F 3 "" H 1350 2350 50  0000 C CNN
+	1    1350 2350
+	-1   0    0    1
+$EndComp
+Wire Wire Line
+	1350 2300 1350 2350
+Connection ~ 1150 2300
+$Comp
+L PWR_FLAG #FLG028
+U 1 1 5757E3F2
+P 1350 2150
+F 0 "#FLG028" H 1350 2245 50  0001 C CNN
+F 1 "PWR_FLAG" H 1350 2330 50  0001 C CNN
+F 2 "" H 1350 2150 50  0000 C CNN
+F 3 "" H 1350 2150 50  0000 C CNN
+	1    1350 2150
+	1    0    0    -1
+$EndComp
+Wire Wire Line
+	1350 2200 1350 2150
+Connection ~ 1150 2200
+$Comp
+L PWR_FLAG #FLG029
+U 1 1 5757E97C
+P 1350 1500
+F 0 "#FLG029" H 1350 1595 50  0001 C CNN
+F 1 "PWR_FLAG" H 1350 1680 50  0001 C CNN
+F 2 "" H 1350 1500 50  0000 C CNN
+F 3 "" H 1350 1500 50  0000 C CNN
+	1    1350 1500
+	1    0    0    -1
+$EndComp
+Wire Wire Line
+	1350 1550 1350 1500
+Connection ~ 1150 1550
 $EndSCHEMATC
