File: 1.3-laboratorio/projetos/ponta-de-prova-logica/ponta-de-prova-logica/ponta-de-prova-logica.sch (KiCad schematic (older format))
At the start: 40 parts

Commit message: Ajustes.
Parts:
- added W?: TEST_1P, symbol TEST_1P
- HIGH, LOW, PULSE: symbol LED -> LED-RESCUE-ponta-de-prova-logica
- U? (x2): symbol LM319 -> LM319-RESCUE-ponta-de-prova-logica
Connections:
- net at 10k.2: now also W?.1
Changed lines of the file:
@@
 EESchema Schematic File Version 2
+LIBS:ponta-de-prova-logica-rescue
 LIBS:power
 LIBS:device
 LIBS:switches
 LIBS:relays
-LIBS:motors
 LIBS:transistors
 LIBS:conn
@@
 LIBS:contrib
 LIBS:valves
+LIBS:ponta-de-prova-logica-cache
 EELAYER 25 0
 EELAYER END
@@
 $EndComp
 $Comp
-L LM319 U?
+L LM319-RESCUE-ponta-de-prova-logica U?
 U 1 1 5B73B4DB
 P 3950 2450
@@
 $EndComp
 $Comp
-L LM319 U?
+L LM319-RESCUE-ponta-de-prova-logica U?
 U 2 1 5B73B621
 P 3950 3550
@@
 $EndComp
 $Comp
-L LED HIGH
+L LED-RESCUE-ponta-de-prova-logica HIGH
 U 1 1 5B73D760
 P 4350 1850
@@
 $EndComp
 $Comp
-L LED LOW
+L LED-RESCUE-ponta-de-prova-logica LOW
 U 1 1 5B73D93F
 P 4350 2950
@@
 $EndComp
 $Comp
-L LED PULSE
+L LED-RESCUE-ponta-de-prova-logica PULSE
 U 1 1 5B746AC3
 P 8500 2300
@@
 	9050 1650 9050 1550
 Connection ~ 8750 1650
+$Comp
+L TEST_1P W?
+U 1 1 5BBEAAFC
+P 2900 3000
+F 0 "W?" H 2900 3270 50  0000 C CNN
+F 1 "TEST_1P" H 2900 3200 50  0000 C CNN
+F 2 "" H 3100 3000 50  0000 C CNN
+F 3 "" H 3100 3000 50  0000 C CNN
+	1    2900 3000
+	1    0    0    -1
+$EndComp
+Wire Wire Line
+	2900 3000 3000 3000
 $EndSCHEMATC

Commit message: Atualização da ponta de prova lógica
Parts:
- removed HIGH, LOW, PULSE: LED, symbol LED-RESCUE-ponta-de-prova-logica
- added 10nF: C, symbol C
- added 390k: R, symbol R
- added D? (x3): LED_ALT, symbol LED_ALT
- gave numbers to parts that had none: 1
Connections:
- net labels added: 39%, 77%, CMOS, TTL
- wire segments 110 -> 115
Changed lines of the file:
@@
 EESchema Schematic File Version 2
-LIBS:ponta-de-prova-logica-rescue
 LIBS:power
 LIBS:device
 LIBS:switches
 LIBS:relays
+LIBS:motors
 LIBS:transistors
 LIBS:conn
@@
 L GND #PWR?
 U 1 1 5B73A64F
-P 2500 4150
-F 0 "#PWR?" H 2500 3900 50  0001 C CNN
-F 1 "GND" H 2500 4000 50  0000 C CNN
-F 2 "" H 2500 4150 50  0001 C CNN
-F 3 "" H 2500 4150 50  0001 C CNN
-	1    2500 4150
+P 2500 4650
+F 0 "#PWR?" H 2500 4400 50  0001 C CNN
+F 1 "GND" H 2500 4500 50  0000 C CNN
+F 2 "" H 2500 4650 50  0001 C CNN
+F 3 "" H 2500 4650 50  0001 C CNN
+	1    2500 4650
 	1    0    0    -1
 $EndComp
@@
 $EndComp
 $Comp
-L SW_DPDT_x2 SW?
+L SW_DPDT_x2 CMOS
 U 1 1 5B73BAC2
 P 2950 2350
-F 0 "SW?" H 2950 2520 50  0000 C CNN
+F 0 "CMOS" H 2950 2520 50  0001 C CNN
 F 1 "SW_DPDT_x2" H 2950 2150 50  0001 C CNN
 F 2 "" H 2950 2350 50  0001 C CNN
@@
 U 1 1 5B73BBBC
 P 2950 3500
-F 0 "SW?" H 2950 3670 50  0000 C CNN
+F 0 "SW?" H 2950 3670 50  0001 C CNN
 F 1 "SW_DPDT_x2" H 2950 3300 50  0001 C CNN
 F 2 "" H 2950 3500 50  0001 C CNN
@@
 $EndComp
 $Comp
-L LED-RESCUE-ponta-de-prova-logica HIGH
-U 1 1 5B73D760
-P 4350 1850
-F 0 "HIGH" H 4350 1950 50  0000 C CNN
-F 1 "LED" H 4350 1750 50  0000 C CNN
-F 2 "" H 4350 1850 50  0001 C CNN
-F 3 "" H 4350 1850 50  0001 C CNN
-	1    4350 1850
-	0    -1   -1   0
-$EndComp
-$Comp
-L LED-RESCUE-ponta-de-prova-logica LOW
-U 1 1 5B73D93F
-P 4350 2950
-F 0 "LOW" H 4350 3050 50  0000 C CNN
-F 1 "LED" H 4350 2850 50  0000 C CNN
-F 2 "" H 4350 2950 50  0001 C CNN
-F 3 "" H 4350 2950 50  0001 C CNN
-	1    4350 2950
-	0    -1   -1   0
-$EndComp
-$Comp
 L R 470R
 U 1 1 5B73DD12
@@
 Connection ~ 2500 4100
 Wire Wire Line
-	3500 4050 3500 4100
+	3500 4050 3500 4200
 Connection ~ 3500 4100
 Wire Wire Line
@@
 Connection ~ 2500 3700
 Wire Wire Line
-	2750 3400 2750 3300
-Wire Wire Line
-	2750 3300 2500 3300
+	2750 3300 2750 3400
+Wire Wire Line
+	2250 3300 2750 3300
 Connection ~ 2500 3300
 Wire Wire Line
@@
 Connection ~ 2500 2600
 Wire Wire Line
-	2750 2250 2750 2200
-Wire Wire Line
-	2750 2200 2500 2200
+	2750 2200 2750 2250
+Wire Wire Line
+	2250 2200 2750 2200
 Connection ~ 2500 2200
 Wire Wire Line
@@
 Connection ~ 3900 2900
 Wire Wire Line
-	3900 4100 3900 3950
-Wire Wire Line
-	2500 4100 3900 4100
+	3900 4550 3900 3950
 Wire Wire Line
 	4350 4550 4350 4700
@@
 $EndComp
 $Comp
-L LED-RESCUE-ponta-de-prova-logica PULSE
-U 1 1 5B746AC3
-P 8500 2300
-F 0 "PULSE" H 8500 2400 50  0000 C CNN
-F 1 "LED" H 8500 2200 50  0000 C CNN
-F 2 "" H 8500 2300 50  0001 C CNN
-F 3 "" H 8500 2300 50  0001 C CNN
-	1    8500 2300
-	0    -1   -1   0
-$EndComp
-$Comp
 L CP 470nF
 U 1 1 5B746D19
@@
 Wire Wire Line
 	2900 3000 3000 3000
+$Comp
+L R 390k
+U 1 1 5BBE97D6
+P 3500 4350
+F 0 "390k" V 3580 4350 50  0000 C CNN
+F 1 "R" V 3500 4350 50  0000 C CNN
+F 2 "" V 3430 4350 50  0001 C CNN
+F 3 "" H 3500 4350 50  0001 C CNN
+	1    3500 4350
+	1    0    0    -1
+$EndComp
+Wire Wire Line
+	3500 4500 3500 4550
+Connection ~ 3500 4550
+Wire Wire Line
+	2500 4100 2500 4650
+Connection ~ 2500 4550
+$Comp
+L C 10nF
+U 1 1 5BBEA261
+P 3200 4200
+F 0 "10nF" H 3225 4300 50  0000 L CNN
+F 1 "C" H 3225 4100 50  0000 L CNN
+F 2 "" H 3238 4050 50  0001 C CNN
+F 3 "" H 3200 4200 50  0001 C CNN
+	1    3200 4200
+	1    0    0    -1
+$EndComp
+Wire Wire Line
+	3200 4050 3200 3700
+Wire Wire Line
+	3200 3700 3500 3700
+Connection ~ 3500 3700
+Wire Wire Line
+	3200 4350 3200 4550
+Connection ~ 3200 4550
+$Comp
+L LED_ALT D?
+U 1 1 5BBEACC7
+P 4350 2950
+F 0 "D?" H 4350 3050 50  0000 C CNN
+F 1 "LED_ALT" H 4350 2850 50  0000 C CNN
+F 2 "" H 4350 2950 50  0001 C CNN
+F 3 "" H 4350 2950 50  0001 C CNN
+	1    4350 2950
+	0    -1   -1   0
+$EndComp
+$Comp
+L LED_ALT D?
+U 1 1 5BBEB02F
+P 4350 1850
+F 0 "D?" H 4350 1950 50  0000 C CNN
+F 1 "LED_ALT" H 4350 1750 50  0000 C CNN
+F 2 "" H 4350 1850 50  0001 C CNN
+F 3 "" H 4350 1850 50  0001 C CNN
+	1    4350 1850
+	0    -1   -1   0
+$EndComp
+$Comp
+L LED_ALT D?
+U 1 1 5BBEB0CE
+P 8500 2300
+F 0 "D?" H 8500 2400 50  0000 C CNN
+F 1 "LED_ALT" H 8500 2200 50  0000 C CNN
+F 2 "" H 8500 2300 50  0001 C CNN
+F 3 "" H 8500 2300 50  0001 C CNN
+	1    8500 2300
+	0    -1   -1   0
+$EndComp
+Wire Wire Line
+	2500 4550 3900 4550
+Text GLabel 2250 3300 0    60   Input ~ 0
+39%
+Text GLabel 2250 2200 0    60   Input ~ 0
+77%
+Text Label 2850 2200 0    60   ~ 0
+CMOS
+Text Label 2900 2550 0    60   ~ 0
+TTL
+Text Label 2850 3350 0    60   ~ 0
+CMOS
+Text Label 2900 3700 0    60   ~ 0
+TTL
 $EndSCHEMATC
