File: 1.3-laboratorio/projetos/ponta-de-prova-logica/ponta-de-prova-logica/ponta-de-prova-logica-simplificada/ponta-de-prova-logica-simplificada.sch (KiCad schematic (older format))
At the start: 18 parts, among them J1 TEST PROBE, J2 Conn_01x02, U1 LM319

Commit message: Correção do arquivo PCB
Parts:
- C1: footprint Capacitors_THT:C_Disc_D5.0mm_W2.5mm_P2.50mm -> Capacitors_THT:C_Disc_D5.0mm_W2.5mm_P5.00mm
- D1, D2: footprint LEDs:LED_D1.8mm_W1.8mm_H2.4mm_Horizontal_O1.27mm_Z1.6mm -> LEDs:LED_D4.0mm
- J2: footprint TerminalBlocks_Phoenix:TerminalBlock_Phoenix_MKDS1.5-2pol -> Connectors_Terminal_Blocks:TerminalBlock_Altech_AK300-2_P5.00mm
Changed lines of the file:
@@
 F 0 "D1" H 4350 2050 50  0001 C CNN
 F 1 "LED HIGH" V 4350 1700 50  0000 C CNN
-F 2 "LEDs:LED_D1.8mm_W1.8mm_H2.4mm_Horizontal_O1.27mm_Z1.6mm" H 4350 1950 50  0001 C CNN
+F 2 "LEDs:LED_D4.0mm" H 4350 1950 50  0001 C CNN
 F 3 "" H 4350 1950 50  0001 C CNN
 	1    4350 1950
@@
 F 0 "D2" H 4350 3350 50  0001 C CNN
 F 1 "LED LOW" V 4350 3000 50  0000 C CNN
-F 2 "LEDs:LED_D1.8mm_W1.8mm_H2.4mm_Horizontal_O1.27mm_Z1.6mm" H 4350 3250 50  0001 C CNN
+F 2 "LEDs:LED_D4.0mm" H 4350 3250 50  0001 C CNN
 F 3 "" H 4350 3250 50  0001 C CNN
 	1    4350 3250
@@
 F 0 "C1" H 2975 4700 50  0000 L CNN
 F 1 "10nF" H 2975 4500 50  0000 L CNN
-F 2 "Capacitors_THT:C_Disc_D5.0mm_W2.5mm_P2.50mm" H 2988 4450 50  0001 C CNN
+F 2 "Capacitors_THT:C_Disc_D5.0mm_W2.5mm_P5.00mm" H 2988 4450 50  0001 C CNN
 F 3 "" H 2950 4600 50  0001 C CNN
 	1    2950 4600
@@
 F 0 "J2" H 1100 1500 50  0000 C CNN
 F 1 "Conn_01x02" H 1100 1200 50  0000 C CNN
-F 2 "TerminalBlocks_Phoenix:TerminalBlock_Phoenix_MKDS1.5-2pol" H 1100 1400 50  0001 C CNN
+F 2 "Connectors_Terminal_Blocks:TerminalBlock_Altech_AK300-2_P5.00mm" H 1100 1400 50  0001 C CNN
 F 3 "" H 1100 1400 50  0001 C CNN
 	1    1100 1400
