File: 2-provas/imagens-fontes/kicad/2019-an-p1/2019-an-p1.sch (KiCad schematic (older format))
At the start: 16 parts

Commit message: Circuitos da prova.
Parts:
- added D1, D?: LED, symbol Device:LED_ALT
- added I0, I?: 1A, symbol simbolos-personalizados:fonte_corrente
- added If, Is: seta_corrente, symbol simbolos-personalizados:seta_corrente
- added R: R_US, symbol Device:R_US
- added R1: 10R, symbol Device:R_US
- added R1: 1,5R, symbol Device:R_US
- added R1: 3k3, symbol Device:R_US
- added R2: 5R, symbol Device:R_US
- added R2, R3 (x2), R? (x2): 2R, symbol Device:R_US
- added R2: 5k6, symbol Device:R_US
- added R4: 6R, symbol Device:R_US
- added V1: 5V, symbol Device:Battery_Cell
- added V1, V2: 12V, symbol Device:Battery_Cell
- added V1: 20V, symbol Device:Battery_Cell
- added V2: 4V, symbol Device:Battery_Cell
- added V3: 3V, symbol Device:Battery_Cell
- added Vf: seta_tensao, symbol simbolos-personalizados:seta_tensao
- added Vs: TestPoint, symbol Connector:TestPoint
Connections:
- new net: R1.1, V1.1 (+)
- new net: V1.2 (-), V2.1 (+), V3.2 (-)
- new net: R2.1, V2.2 (-)
- new net: R3.1, V3.1 (+)
- new net: I0.1 (+), R1.2, R2.2, R3.2, R4.2
- new net: I0.2 (-), R4.1
- new net: R.2, V1.1 (+)
- new net: D1.1 (K), V1.2 (-)
- new net: D1.2 (A), R.1
- new net: R1.2, V1.1 (+)
- new net: R2.1, V1.2 (-), V2.2 (-)
- new net: R1.1, R2.2, R3.2
- new net: R3.1, V2.1 (+)
- new net: I?.1 (+), R?.2, R?.2
- new net: I?.2 (-), R?.1, R?.1
- new net: R1.1, R2.2, Vs.1
- new net +12V: R1.2
- new net Earth: R2.1
Other:
- note added: "0,08W"
- note added: "112W"
- note added: "47W"
- note added: "67,3W"
- note added: "Vf = 3,0V\nIf = 20 mA\nIf(mín) = 15 mA (*)\nIf(máx) = 25mA\n\n(*) Para brilho mínimo desejável."
- moved on the sheet: R1, R2, R3, V1, V2, V3

Commit message: Finalizada a prova.
Parts:
- added I: seta_corrente, symbol simbolos-personalizados:seta_corrente
- gave numbers to parts that had none: 3
Other:
- moved on the sheet: R1, R2, Vs
Changed lines of the file:
@@
 0,08W
 $Comp
-L simbolos-personalizados:fonte_corrente I?
+L simbolos-personalizados:fonte_corrente Icc
 U 1 1 5D93E34B
 P 7250 2650
-F 0 "I?" V 7100 2650 50  0000 C CNN
-F 1 "1A" V 7400 2650 50  0000 C CNN
+F 0 "Icc" H 7100 2750 50  0000 C CNN
+F 1 "1A" H 7400 2650 50  0000 C CNN
 F 2 "" V 7250 2650 50  0001 C CNN
 F 3 "" V 7250 2650 50  0001 C CNN
@@
 $EndComp
 $Comp
-L Device:R_US R?
+L Device:R_US R1
 U 1 1 5D93EEC7
 P 7650 2650
-F 0 "R?" H 7525 2700 50  0000 C CNN
+F 0 "R1" H 7525 2700 50  0000 C CNN
 F 1 "2R" H 7525 2600 50  0000 C CNN
 F 2 "" V 7690 2640 50  0001 C CNN
@@
 $EndComp
 $Comp
-L Device:R_US R?
+L Device:R_US R2
 U 1 1 5D93EF4D
 P 8050 2650
-F 0 "R?" H 7925 2700 50  0000 C CNN
+F 0 "R2" H 7925 2700 50  0000 C CNN
 F 1 "2R" H 7925 2600 50  0000 C CNN
 F 2 "" V 8090 2640 50  0001 C CNN
@@
 L power:+12V #PWR?
 U 1 1 5D946920
-P 7600 3400
-F 0 "#PWR?" H 7600 3250 50  0001 C CNN
-F 1 "+12V" H 7615 3573 50  0000 C CNN
-F 2 "" H 7600 3400 50  0001 C CNN
-F 3 "" H 7600 3400 50  0001 C CNN
-	1    7600 3400
+P 7600 3550
+F 0 "#PWR?" H 7600 3400 50  0001 C CNN
+F 1 "+12V" H 7615 3723 50  0000 C CNN
+F 2 "" H 7600 3550 50  0001 C CNN
+F 3 "" H 7600 3550 50  0001 C CNN
+	1    7600 3550
 	1    0    0    -1
 $EndComp
@@
 L Device:R_US R1
 U 1 1 5D946978
-P 7600 3600
-F 0 "R1" H 7475 3650 50  0000 C CNN
-F 1 "3k3" H 7475 3550 50  0000 C CNN
-F 2 "" V 7640 3590 50  0001 C CNN
-F 3 "~" H 7600 3600 50  0001 C CNN
-	1    7600 3600
+P 7600 3750
+F 0 "R1" H 7475 3800 50  0000 C CNN
+F 1 "3k3" H 7475 3700 50  0000 C CNN
+F 2 "" V 7640 3740 50  0001 C CNN
+F 3 "~" H 7600 3750 50  0001 C CNN
+	1    7600 3750
 	-1   0    0    1
 $EndComp
@@
 L Device:R_US R2
 U 1 1 5D9469F8
-P 7600 4000
-F 0 "R2" H 7475 4050 50  0000 C CNN
-F 1 "5k6" H 7475 3950 50  0000 C CNN
-F 2 "" V 7640 3990 50  0001 C CNN
-F 3 "~" H 7600 4000 50  0001 C CNN
-	1    7600 4000
+P 7600 4150
+F 0 "R2" H 7475 4200 50  0000 C CNN
+F 1 "5k6" H 7475 4100 50  0000 C CNN
+F 2 "" V 7640 4140 50  0001 C CNN
+F 3 "~" H 7600 4150 50  0001 C CNN
+	1    7600 4150
 	-1   0    0    1
 $EndComp
@@
 L power:Earth #PWR?
 U 1 1 5D947348
-P 7600 4200
-F 0 "#PWR?" H 7600 3950 50  0001 C CNN
-F 1 "Earth" H 7600 4050 50  0001 C CNN
-F 2 "" H 7600 4200 50  0001 C CNN
-F 3 "~" H 7600 4200 50  0001 C CNN
-	1    7600 4200
+P 7600 4350
+F 0 "#PWR?" H 7600 4100 50  0001 C CNN
+F 1 "Earth" H 7600 4200 50  0001 C CNN
+F 2 "" H 7600 4350 50  0001 C CNN
+F 3 "~" H 7600 4350 50  0001 C CNN
+	1    7600 4350
 	1    0    0    -1
 $EndComp
 Wire Wire Line
-	7600 3400 7600 3450
+	7600 3550 7600 3600
 Wire Wire Line
-	7600 3750 7600 3800
+	7600 3900 7600 3950
 Wire Wire Line
-	7600 4150 7600 4200
+	7600 4300 7600 4350
 Wire Wire Line
-	7600 3800 7800 3800
-Connection ~ 7600 3800
+	7600 3950 7800 3950
+Connection ~ 7600 3950
 Wire Wire Line
-	7600 3800 7600 3850
+	7600 3950 7600 4000
 $Comp
 L Connector:TestPoint Vs
 U 1 1 5D94F393
-P 7800 3800
-F 0 "Vs" V 7800 3988 50  0000 L CNN
-F 1 "TestPoint" V 7845 3988 50  0001 L CNN
-F 2 "" H 8000 3800 50  0001 C CNN
-F 3 "~" H 8000 3800 50  0001 C CNN
-	1    7800 3800
+P 7800 3950
+F 0 "Vs" V 7800 4138 50  0000 L CNN
+F 1 "TestPoint" V 7845 4138 50  0001 L CNN
+F 2 "" H 8000 3950 50  0001 C CNN
+F 3 "~" H 8000 3950 50  0001 C CNN
+	1    7800 3950
 	0    1    1    0
 $EndComp
+$Comp
+L simbolos-personalizados:seta_corrente I
+U 1 1 5D969C9C
+P 3900 1900
+F 0 "I" H 3999 1993 50  0000 C CNN
+F 1 "seta_corrente" H 4000 1850 50  0001 C CNN
+F 2 "" H 3900 1900 50  0001 C CNN
+F 3 "" H 3900 1900 50  0001 C CNN
+	1    3900 1900
+	1    0    0    -1
+$EndComp
 $EndSCHEMATC
