File: 1.3-laboratorio/projetos/depuracao-circuitos/circuito-01/circuito-01-com-defeito.kicad_pcb (KiCad board)
At the start: 2 copper layers, 76.2 x 54.6 mm, 26 parts, among them J1 Conn_01x07_Male, J2 Conn_01x07_Male, J3 Conn_01x07_Male, J4 Conn_01x07_Male, J5 Conn_01x07_Male, J6 Conn_01x07_Male, J7 Conn_01x05, J8 Conn_01x05, P1 CONN_01X02, SW1 SW_DIP_x04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

Commit message: Do circuito para depuração 01, elaborada a versão com defeito.
Parts:
- D1: value LED_VD -> LED_ALT
Connections:
- J6 pad 2: /U2-08 -> /U3-09
- J8 pad 5: Net-(J8-Pad5) -> /U2-02
- U3 pad 9: /U2-08 -> /U3-09
Routing:
- net GND: track 0.00 -> 15.2 mm
- net /U2-08: track 36.2 -> 24.5 mm
- net /U2-02: track 74.1 -> 84.1 mm
- net /U3-09: track 0.00 -> 3.81 mm
Other:
- board text added: "Circuito 01 (com defeito)"
- board text added: "JP12"
- board text removed: "Circuito 01 (sem defeito)"
Changed lines of the file:
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@@
   (general
     (thickness 1.6)
-    (drawings 43)
-    (tracks 225)
+    (drawings 44)
+    (tracks 229)
     (zones 0)
     (modules 26)
@@
     (visible_elements 7FFFFFFF)
     (pcbplotparams
-      (layerselection 0x00020_ffffffff)
+      (layerselection 0x01020_ffffffff)
       (usegerberextensions false)
       (usegerberattributes false)
@@
       (psa4output false)
       (plotreference true)
-      (plotvalue true)
+      (plotvalue false)
       (plotinvisibletext false)
       (padsonsilk false)
@@
       (drillshape 0)
       (scaleselection 1)
-      (outputdirectory ""))
+      (outputdirectory "gerber-com-defeito/"))
   )
   (net 0 "")
@@
   (net 26 /U3-02)
   (net 27 /U3-01)
-  (net 28 "Net-(J8-Pad5)")
+  (net 28 /U3-09)
   (net_class Default "Esta é a classe de net default."
     (clearance 0.508)
@@
     (add_net /U3-05)
     (add_net /U3-06)
+    (add_net /U3-09)
     (add_net /U3-10)
     (add_net /U3-11)
@@
     (add_net GND)
     (add_net "Net-(D1-Pad2)")
-    (add_net "Net-(J8-Pad5)")
   )
   (net_class Alimentacao ""
@@
       (effects (font (size 1 1) (thickness 0.15)))
     )
-    (fp_text value LED_VD (at 1.27 3.96 180) (layer F.Fab)
+    (fp_text value LED_ALT (at 1.27 3.96 180) (layer F.Fab)
       (effects (font (size 1 1) (thickness 0.15)))
     )
@@
     (fp_line (start -1.27 -1.27) (end 0.635 -1.27) (layer F.Fab) (width 0.1))
     (pad 5 thru_hole oval (at 0 10.16) (size 3 2) (drill 1) (layers *.Cu *.Mask)
-      (net 28 "Net-(J8-Pad5)"))
+      (net 17 /U2-02))
     (pad 4 thru_hole oval (at 0 7.62) (size 3 2) (drill 1) (layers *.Cu *.Mask)
       (net 12 /U3-10))
@@
       (net 11 /U2-11))
     (pad 2 thru_hole oval (at 0 2.54 270) (size 3 2) (drill 1) (layers *.Cu *.Mask)
-      (net 6 /U2-08))
+      (net 28 /U3-09))
     (pad 3 thru_hole oval (at 0 5.08 270) (size 3 2) (drill 1) (layers *.Cu *.Mask)
       (net 12 /U3-10))
@@
       (net 10 /U3-03))
     (pad 9 thru_hole oval (at 7.62 12.7 90) (size 3 2) (drill 0.9) (layers *.Cu *.Mask)
-      (net 6 /U2-08))
+      (net 28 /U3-09))
     (pad 2 thru_hole oval (at 0 2.54 90) (size 3 2) (drill 0.9) (layers *.Cu *.Mask)
       (net 26 /U3-02))
@@
     (pad 1 thru_hole circle (at 0 0) (size 3.8 3.8) (drill 2.2) (layers *.Cu *.Mask))
   )
+  (gr_text JP12 (at 139.7 107.315) (layer F.SilkS)
+    (effects (font (size 1 1) (thickness 0.15)))
+  )
   (gr_text JP11 (at 139.7 104.775) (layer F.Fab)
     (effects (font (size 1 1) (thickness 0.15)))
@@
     (effects (font (size 1 1) (thickness 0.2)) (justify mirror))
   )
-  (gr_text "Circuito 01\n(sem defeito)" (at 164.465 73.025) (layer F.SilkS)
+  (gr_text "Circuito 01\n(com defeito)" (at 164.465 73.025) (layer F.SilkS)
     (effects (font (size 1 1) (thickness 0.15)))
   )
@@
   (segment (start 163.83 74.93) (end 162.56 73.66) (width 0.5) (layer B.Cu) (net 5))
   (segment (start 176.53 77.47) (end 176.53 81.28) (width 0.5) (layer B.Cu) (net 6) (status 30))
-  (segment (start 173.99 107.95) (end 173.99 104.14) (width 0.5) (layer B.Cu) (net 6) (status 30))
   (via (at 179.07 95.25) (size 2) (drill 0.9) (layers F.Cu B.Cu) (net 6))
   (segment (start 179.07 85.82) (end 179.07 95.25) (width 0.5) (layer B.Cu) (net 6))
   (segment (start 176.53 81.28) (end 176.53 83.28) (width 0.5) (layer B.Cu) (net 6) (status 10))
   (segment (start 176.53 83.28) (end 179.07 85.82) (width 0.5) (layer B.Cu) (net 6))
-  (segment (start 173.99 101.6) (end 173.99 104.14) (width 0.5) (layer B.Cu) (net 6) (status 20))
   (via (at 179.07 100.965) (size 2) (drill 0.9) (layers F.Cu B.Cu) (net 6))
   (segment (start 179.07 95.25) (end 179.07 100.965) (width 0.5) (layer F.Cu) (net 6))
-  (segment (start 174.625 100.965) (end 173.99 101.6) (width 0.5) (layer B.Cu) (net 6))
-  (segment (start 179.07 100.965) (end 174.625 100.965) (width 0.5) (layer B.Cu) (net 6))
   (segment (start 173.99 119.38) (end 173.99 115.57) (width 0.5) (layer B.Cu) (net 7) (status 30))
   (segment (start 171.45 115.57) (end 171.45 119.38) (width 0.5) (layer B.Cu) (net 8) (status 30))
@@
   (segment (start 147.32 103.505) (end 152.420541 103.505) (width 0.5) (layer B.Cu) (net 17))
   (segment (start 152.420541 103.505) (end 160.957539 94.968001) (width 0.5) (layer B.Cu) (net 17))
+  (segment (start 134.08 108.585) (end 147.32 108.585) (width 0.5) (layer F.Cu) (net 1))
+  (segment (start 132.08 108.585) (end 134.08 108.585) (width 0.5) (layer F.Cu) (net 1))
+  (segment (start 134.08 108.585) (end 132.08 108.585) (width 0.5) (layer B.Cu) (net 17))
+  (segment (start 135.255 107.41) (end 134.08 108.585) (width 0.5) (layer B.Cu) (net 17))
+  (segment (start 135.255 104.68) (end 135.255 107.41) (width 0.5) (layer B.Cu) (net 17))
+  (segment (start 134.08 103.505) (end 135.255 104.68) (width 0.5) (layer B.Cu) (net 17))
+  (segment (start 132.08 103.505) (end 134.08 103.505) (width 0.5) (layer B.Cu) (net 17))
+  (segment (start 173.99 107.95) (end 173.99 104.14) (width 0.5) (layer B.Cu) (net 28) (status 30))
   (segment (start 142.24 88.9) (end 142.24 92.71) (width 0.5) (layer B.Cu) (net 18) (status 30))
   (segment (start 136.66 118.11) (end 137.16 118.11) (width 0.5) (layer B.Cu) (net 18) (status 30))
