File: 1.1-teoria/trabalhos/substituicao-p1-2020/substituicao-p1-2020-circuitos/substituicao-p1-2020-circuitos.sch (KiCad schematic (older format))
At the start: 0 parts

Commit message: Sincronização e reestruturação de diretório.
Other:
- note added: "=> Circuitos feitos no Logisim e no Digital. <="
Changed lines of the file:
@@
 Text Notes 850  2300 0    50   ~ 0
 Operações aritméticas em binário, em 1 byte.
+Text Notes 900  2700 0    50   ~ 0
+=> Circuitos feitos no Logisim e no Digital. <=
 $EndSCHEMATC
