File: 1.3-laboratorio/experiencias/imagens-fontes/kicad/painel-digital-e-protoboard/5v-r-led-r-led.sch (KiCad schematic (older format))
At the start: 5 parts

Commit message: Sincronismo.
Parts:
- R1: value 330 -> 270
- R2: value 330 -> 470
Changed lines of the file:
@@
 EESchema Schematic File Version 4
-LIBS:5v-r-led-cache
+LIBS:5v-r-led-r-led-cache
 EELAYER 26 0
 EELAYER END
@@
 P 5550 3400
 F 0 "R1" V 5435 3400 50  0000 C CNN
-F 1 "330" V 5650 3400 50  0000 C CNN
+F 1 "270" V 5650 3400 50  0000 C CNN
 F 2 "" V 5480 3400 50  0001 C CNN
 F 3 "~" H 5550 3400 50  0001 C CNN
@@
 P 6000 3400
 F 0 "R2" V 5885 3400 50  0000 C CNN
-F 1 "330" V 6100 3400 50  0000 C CNN
+F 1 "470" V 6100 3400 50  0000 C CNN
 F 2 "" V 5930 3400 50  0001 C CNN
 F 3 "~" H 6000 3400 50  0001 C CNN
