File: 1.3-laboratorio/experiencias/imagens-fontes/kicad/painel-digital-e-protoboard/5v-r-r-r-led.sch (KiCad schematic (older format))
At the start: 5 parts

Commit message: Sincronismo.
Parts:
- R1, R2, R3: value 330 -> 100
Changed lines of the file:
@@
 EESchema Schematic File Version 4
-LIBS:5v-r-led-cache
+LIBS:5v-r-r-r-led-cache
 EELAYER 26 0
 EELAYER END
@@
 P 5500 2900
 F 0 "R1" V 5385 2900 50  0000 C CNN
-F 1 "330" V 5600 2900 50  0000 C CNN
+F 1 "100" V 5600 2900 50  0000 C CNN
 F 2 "" V 5430 2900 50  0001 C CNN
 F 3 "~" H 5500 2900 50  0001 C CNN
@@
 P 5900 2900
 F 0 "R2" V 5785 2900 50  0000 C CNN
-F 1 "330" V 6000 2900 50  0000 C CNN
+F 1 "100" V 6000 2900 50  0000 C CNN
 F 2 "" V 5830 2900 50  0001 C CNN
 F 3 "~" H 5900 2900 50  0001 C CNN
@@
 P 6300 2900
 F 0 "R3" V 6185 2900 50  0000 C CNN
-F 1 "330" V 6400 2900 50  0000 C CNN
+F 1 "100" V 6400 2900 50  0000 C CNN
 F 2 "" V 6230 2900 50  0001 C CNN
 F 3 "~" H 6300 2900 50  0001 C CNN
