File: 1.3-laboratorio/projetos/dado-digital/dado-digital-simplificado/dado-digital-simplificado.sch (KiCad schematic (older format))
At the start: 25 parts, among them J1 Conn_01x02, SW1 SW_Push, U1 74HC74, U2 74HC74, U3 74HC14, U4 74HC08, U5 CD4511BE, U6 HDSP-7403

Commit message: Esquemático do Dado Digital Simplificado. Falta revisão final.
Parts:
- added C8, C9: 10uF, symbol Device:CP1
- added D1: 1N4148, Diode_THT:D_DO-35_SOD27_P7.62mm_Horizontal, symbol Device:D_ALT
- added R2: 330k, symbol Device:R
- added R3: 10k, symbol Device:R
- added SW1: SW_DPST, symbol Switch:SW_DPST
- C1: renamed from C2; Observação (none) -> Bypass U1
- C2: renamed from C3; Observação (none) -> Bypass U2
- C3: renamed from C4; Observação (none) -> Bypass U3
- C4: renamed from C5; Observação (none) -> Bypass U4
- C5: renamed from C6; Observação (none) -> Bypass U5
- C6: renamed from C7; value CP1 -> 10uF; Value 100nF -> (none)
- C7: renamed from C1; value CP1 -> 1uF; Value 100nF -> (none)
- J1: Observação (none) -> 3 x 1,5V (AA)
- R1: value R -> 10k
- R12: renamed from R9; value 220R -> 330R
- R4: renamed from R10; value R -> 10k
- renumbered U6 to DISP1, R7 to R10, R8 to R11, R2 to R5, R3 to R6, R4 to R7, R5 to R8, R6 to R9, SW1 to SW2
Connections:
- net Earth: now also C1.2, C2.2, C3.2, C4.2, C5.2, DISP1.1 (CC), DISP1.6 (CC), U1.7 (GND), U2.7 (GND), U3.7 (GND), U4.7 (GND), U5.5 (LE/~STROBE), C8.2, C9.2, SW1.2; no longer J1.2 (Pin_2)
- net VCC: now also C1.1, C2.1, C3.1, C4.1, C5.1, R12.1, U1.14 (VCC), U1.4 (~S), U2.14 (VCC), U3.13, U3.14 (VCC), U4.14 (VCC), SW1.4; no longer J1.1 (Pin_1)
- net ck: now also U3.4, R3.1
- net ~HAB_CK: now also D1.1 (K), R2.2
- net ~POR: now also U3.2; no longer U3.4
- net at U1.3 (C): now also U3.8; no longer U3.2
- net ~BI: now reaches U5.4 (~BT)
- net ~BI: now also U3.10
- net DP: now reaches DISP1.7 (DP)
- net DP: now also R12.2; no longer R12.1
- net at C7.1, R1.2, SW2.2: now also U3.9; no longer U3.1
- net at U4.9: now also U3.6; no longer U3.8
- net at U4.6: now also U3.5; no longer U3.9
- net at C6.2, R4.1: now also U3.1; no longer U3.3
- new net: J1.1 (Pin_1), SW1.3
- new net: J1.2 (Pin_2), SW1.1
- new net: C8.1, D1.2 (A), R2.1, U3.11
- new net: C9.1, R3.2, U3.3
- no-connect marks 0 -> 1
Other:
- note added: "7 x 220R"
- note added: "Alimentação"
- note added: "Alimentação de CIs"
- note added: "Bypass dos CIs"
- note added: "Conta-Pára"
- note added: "Contador"
- note added: "Debouncing"
- note added: "Decodificador e Driver"
- note added: "Display"
- note added: "Gerador de clock"
- note added: "Partes Não Utilizadas"
- note added: "Ponto\nDecimal"
- note added: "Power-On Reset"
- note added: "Temporizador"
- moved on the sheet: C1, C2, C3, C4, C5, C6, C7, DISP1, J1, R1, R10, R11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
