File: 1.3-laboratorio/projetos/ponta-de-prova-logica/ponta-de-prova-logica-simplificada/pcb-versoes-anteriores/do-aluno-monitor/Prova_Logica_SMD/Original/ponta-de-prova-logica-simplificada.sch (KiCad schematic (older format))
At the start: 21 parts, among them J1 Conn_01x02, J2 TEST_1P, J3 TEST_1P, SW1 SW_DPDT_x2, U1 LM339

Commit message: Ponta_Logica_SMD_v2
Versao 2 - Projeto Ponta Lógica monitor
Parts:
- U1: footprint Package_DIP:DIP-14_W7.62mm_Socket_LongPads -> Package_SO:SOIC-14_3.9x8.7mm_P1.27mm
Changed lines of the file:
@@
 F 0 "U1" H 7700 4450 50  0000 C CNN
 F 1 "LM339" H 7700 4350 50  0000 C CNN
-F 2 "Package_DIP:DIP-14_W7.62mm_Socket_LongPads" H 7500 4300 50  0001 C CNN
+F 2 "Package_SO:SOIC-14_3.9x8.7mm_P1.27mm" H 7500 4300 50  0001 C CNN
 F 3 "http://www.ti.com/lit/ds/symlink/lm339.pdf" H 7600 4400 50  0001 C CNN
 	1    7550 4200
@@
 F 0 "U1" H 7700 3600 50  0000 C CNN
 F 1 "LM339" H 7700 3500 50  0000 C CNN
-F 2 "Package_DIP:DIP-14_W7.62mm_Socket_LongPads" H 7500 3450 50  0001 C CNN
+F 2 "Package_SO:SOIC-14_3.9x8.7mm_P1.27mm" H 7500 3450 50  0001 C CNN
 F 3 "http://www.ti.com/lit/ds/symlink/lm339.pdf" H 7600 3550 50  0001 C CNN
 	2    7550 3350
@@
 F 0 "U1" H 3850 4600 50  0000 C CNN
 F 1 "LM339" H 3850 4500 50  0000 C CNN
-F 2 "Package_DIP:DIP-14_W7.62mm_Socket_LongPads" H 3650 4450 50  0001 C CNN
+F 2 "Package_SO:SOIC-14_3.9x8.7mm_P1.27mm" H 3650 4450 50  0001 C CNN
 F 3 "http://www.ti.com/lit/ds/symlink/lm339.pdf" H 3750 4550 50  0001 C CNN
 	3    3700 4350
@@
 F 0 "U1" H 3850 5200 50  0000 C CNN
 F 1 "LM339" H 3850 5100 50  0000 C CNN
-F 2 "Package_DIP:DIP-14_W7.62mm_Socket_LongPads" H 3650 5050 50  0001 C CNN
+F 2 "Package_SO:SOIC-14_3.9x8.7mm_P1.27mm" H 3650 5050 50  0001 C CNN
 F 3 "http://www.ti.com/lit/ds/symlink/lm339.pdf" H 3750 5150 50  0001 C CNN
 	4    3700 4950
@@
 F 0 "U1" H 7508 3396 50  0001 L CNN
 F 1 "LM339" H 7508 3305 50  0001 L CNN
-F 2 "Package_DIP:DIP-14_W7.62mm_Socket_LongPads" H 7500 3450 50  0001 C CNN
+F 2 "Package_SO:SOIC-14_3.9x8.7mm_P1.27mm" H 7500 3450 50  0001 C CNN
 F 3 "http://www.ti.com/lit/ds/symlink/lm339.pdf" H 7600 3550 50  0001 C CNN
 	5    7550 3350
