File: 1.3-laboratorio/projetos/cronometros/cronometro-conta-para-zera/driver-displays.sch (KiCad schematic (older format))
At the start: 33 parts

Commit message: Concluído esquemático do Cronômetro Digital Didático. Faltam revisões.
Parts:
- added R?: 270R, symbol Device:R
- added U12, U13, U14: HDSP-7803, Display_7Segment:HDSP-7801, symbol Display_Character:HDSP-7803
- gave numbers to parts that had none: 33
Connections:
- wire segments 114 -> 137
Other:
- moved on the sheet: R10, R11, R12, R13, R14, R15, R16, R17, R18, R19, R20, R21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

Commit message: Concluído esquemático do Cronômetro Digital Didático. Faltam revisões.
Parts:
- gave numbers to parts that had none: 1
Changed lines of the file:
@@
 P 7150 800
 AR Path="/5FEFC556" Ref="#PWR?"  Part="1"
-AR Path="/5FA6DD7C/5FEFC556" Ref="#PWR?"  Part="1"
-F 0 "#PWR?" H 7150 650 50  0001 C CNN
+AR Path="/5FA6DD7C/5FEFC556" Ref="#PWR027"  Part="1"
+F 0 "#PWR027" H 7150 650 50  0001 C CNN
 F 1 "VCC" H 7165 973 50  0000 C CNN
 F 2 "" H 7150 800 50  0001 C CNN
@@
 $EndComp
 $Comp
-L Device:R R?
+L Device:R R6
 U 1 1 5FEFC958
 P 7150 1000
-F 0 "R?" V 7150 1000 50  0000 C CNN
+F 0 "R6" V 7150 1000 50  0000 C CNN
 F 1 "270R" V 7034 1000 50  0001 C CNN
 F 2 "" V 7080 1000 50  0001 C CNN

Commit message: Adicionado PWR_FLAG no projeto do cronômetro. Datasheets de componentes.
Parts:
- U10, U7, U8, U9: symbol eec:CD4511BNSR -> cronometro-conta-para-zera-rescue:CD4511BNSR-eec
Changed lines of the file:
@@
 $EndDescr
 $Comp
-L eec:CD4511BNSR U?
+L cronometro-conta-para-zera-rescue:CD4511BNSR-eec U?
 U 1 1 5FA79889
 P 4150 950
@@
 DS3
 $Comp
-L eec:CD4511BNSR U?
+L cronometro-conta-para-zera-rescue:CD4511BNSR-eec U?
 U 1 1 5FA798D0
 P 4150 4450
@@
 	2800 5050 3800 5050
 $Comp
-L eec:CD4511BNSR U?
+L cronometro-conta-para-zera-rescue:CD4511BNSR-eec U?
 U 1 1 5FA79917
 P 4150 2700
@@
 	2800 3300 3800 3300
 $Comp
-L eec:CD4511BNSR U?
+L cronometro-conta-para-zera-rescue:CD4511BNSR-eec U?
 U 1 1 5FA7995E
 P 4200 6200

Commit message: Em elaboração a PCI. Ajustes no esquemático foram feitos.
Parts:
- R10, R11, R12, R13, R14, R15, R16, R17, R18, R19, R20, R21, R22, R23, R24, R25, R26, R27, R28, R29, R30, R31, R32, R33, R34, R6, R7, R8, R9: footprint (none) -> Resistor_THT:R_Axial_DIN0204_L3.6mm_D1.6mm_P7.62mm_Horizontal
- U10, U7, U8, U9: footprint Texas_Instruments-CD4511BNSR-* -> Package_DIP:DIP-16_W7.62mm_Socket_LongPads
Changed lines of the file:
@@
 Sheet 2 2
 Title "Cronômetro Digital Didático"
-Date "2020-10-13"
+Date "2020-10-14"
 Rev "0.0"
 Comp "Fundamentos de Circuitos Digitais e Analógicos"
 Comment1 "Décimos de segundo a unidades de minuto."
 Comment2 "Todos resistores de 1/8W, 5% de tolerância."
-Comment3 ""
+Comment3 "CC BY 4.0 (https://creativecommons.org/licenses/by/4.0/)"
 Comment4 ""
 $EndDescr
@@
 F 0 "U7" H 4750 1215 50  0000 C CNN
 F 1 "CD4511BNSR" H 4750 1124 50  0000 C CNN
-F 2 "Texas_Instruments-CD4511BNSR-*" H 4150 1350 50  0001 L CNN
+F 2 "Package_DIP:DIP-16_W7.62mm_Socket_LongPads" H 4150 1350 50  0001 L CNN
 F 3 "http://www.ti.com/general/docs/lit/getliterature.tsp?genericPartNumber=CD4511B&fileType=pdf" H 4150 1450 50  0001 L CNN
 F 4 "Manufacturer URL" H 4150 1550 50  0001 L CNN "Component Link 1 Description"
@@
 F 0 "U9" H 4750 4715 50  0000 C CNN
 F 1 "CD4511BNSR" H 4750 4624 50  0000 C CNN
-F 2 "Texas_Instruments-CD4511BNSR-*" H 4150 4850 50  0001 L CNN
+F 2 "Package_DIP:DIP-16_W7.62mm_Socket_LongPads" H 4150 4850 50  0001 L CNN
 F 3 "http://www.ti.com/general/docs/lit/getliterature.tsp?genericPartNumber=CD4511B&fileType=pdf" H 4150 4950 50  0001 L CNN
 F 4 "Manufacturer URL" H 4150 5050 50  0001 L CNN "Component Link 1 Description"
@@
 F 0 "U8" H 4750 2965 50  0000 C CNN
 F 1 "CD4511BNSR" H 4750 2874 50  0000 C CNN
-F 2 "Texas_Instruments-CD4511BNSR-*" H 4150 3100 50  0001 L CNN
+F 2 "Package_DIP:DIP-16_W7.62mm_Socket_LongPads" H 4150 3100 50  0001 L CNN
 F 3 "http://www.ti.com/general/docs/lit/getliterature.tsp?genericPartNumber=CD4511B&fileType=pdf" H 4150 3200 50  0001 L CNN
 F 4 "Manufacturer URL" H 4150 3300 50  0001 L CNN "Component Link 1 Description"
@@
 F 0 "U10" H 4800 6465 50  0000 C CNN
 F 1 "CD4511BNSR" H 4800 6374 50  0000 C CNN
-F 2 "Texas_Instruments-CD4511BNSR-*" H 4200 6600 50  0001 L CNN
+F 2 "Package_DIP:DIP-16_W7.62mm_Socket_LongPads" H 4200 6600 50  0001 L CNN
 F 3 "http://www.ti.com/general/docs/lit/getliterature.tsp?genericPartNumber=CD4511B&fileType=pdf" H 4200 6700 50  0001 L CNN
 F 4 "Manufacturer URL" H 4200 6800 50  0001 L CNN "Component Link 1 Description"
@@
 F 0 "R7" V 5500 950 50  0000 C CNN
 F 1 "270R" V 5384 950 50  0001 C CNN
-F 2 "" V 5430 950 50  0001 C CNN
+F 2 "Resistor_THT:R_Axial_DIN0204_L3.6mm_D1.6mm_P7.62mm_Horizontal" V 5430 950 50  0001 C CNN
 F 3 "~" H 5500 950 50  0001 C CNN
 	1    5500 950
@@
 F 0 "R8" V 5500 1050 50  0000 C CNN
 F 1 "270R" V 5384 1050 50  0001 C CNN
-F 2 "" V 5430 1050 50  0001 C CNN
+F 2 "Resistor_THT:R_Axial_DIN0204_L3.6mm_D1.6mm_P7.62mm_Horizontal" V 5430 1050 50  0001 C CNN
 F 3 "~" H 5500 1050 50  0001 C CNN
 	1    5500 1050
@@
 F 0 "R9" V 5500 1150 50  0000 C CNN
 F 1 "270R" V 5384 1150 50  0001 C CNN
-F 2 "" V 5430 1150 50  0001 C CNN
+F 2 "Resistor_THT:R_Axial_DIN0204_L3.6mm_D1.6mm_P7.62mm_Horizontal" V 5430 1150 50  0001 C CNN
 F 3 "~" H 5500 1150 50  0001 C CNN
 	1    5500 1150
@@
 F 0 "R10" V 5500 1250 50  0000 C CNN
 F 1 "270R" V 5384 1250 50  0001 C CNN
-F 2 "" V 5430 1250 50  0001 C CNN
+F 2 "Resistor_THT:R_Axial_DIN0204_L3.6mm_D1.6mm_P7.62mm_Horizontal" V 5430 1250 50  0001 C CNN
 F 3 "~" H 5500 1250 50  0001 C CNN
 	1    5500 1250
@@
 F 0 "R11" V 5500 1350 50  0000 C CNN
 F 1 "270R" V 5384 1350 50  0001 C CNN
-F 2 "" V 5430 1350 50  0001 C CNN
+F 2 "Resistor_THT:R_Axial_DIN0204_L3.6mm_D1.6mm_P7.62mm_Horizontal" V 5430 1350 50  0001 C CNN
 F 3 "~" H 5500 1350 50  0001 C CNN
 	1    5500 1350
@@
 F 0 "R12" V 5500 1450 50  0000 C CNN
 F 1 "270R" V 5384 1450 50  0001 C CNN
-F 2 "" V 5430 1450 50  0001 C CNN
+F 2 "Resistor_THT:R_Axial_DIN0204_L3.6mm_D1.6mm_P7.62mm_Horizontal" V 5430 1450 50  0001 C CNN
 F 3 "~" H 5500 1450 50  0001 C CNN
 	1    5500 1450
@@
 F 0 "R13" V 5500 1550 50  0000 C CNN
 F 1 "270R" V 5384 1550 50  0001 C CNN
-F 2 "" V 5430 1550 50  0001 C CNN
+F 2 "Resistor_THT:R_Axial_DIN0204_L3.6mm_D1.6mm_P7.62mm_Horizontal" V 5430 1550 50  0001 C CNN
 F 3 "~" H 5500 1550 50  0001 C CNN
 	1    5500 1550
@@
 F 0 "R14" V 5500 2700 50  0000 C CNN
 F 1 "270R" V 5384 2700 50  0001 C CNN
-F 2 "" V 5430 2700 50  0001 C CNN
+F 2 "Resistor_THT:R_Axial_DIN0204_L3.6mm_D1.6mm_P7.62mm_Horizontal" V 5430 2700 50  0001 C CNN
 F 3 "~" H 5500 2700 50  0001 C CNN
 	1    5500 2700
@@
 F 0 "R15" V 5500 2800 50  0000 C CNN
 F 1 "270R" V 5384 2800 50  0001 C CNN
-F 2 "" V 5430 2800 50  0001 C CNN
+F 2 "Resistor_THT:R_Axial_DIN0204_L3.6mm_D1.6mm_P7.62mm_Horizontal" V 5430 2800 50  0001 C CNN
 F 3 "~" H 5500 2800 50  0001 C CNN
 	1    5500 2800
@@
 F 0 "R16" V 5500 2900 50  0000 C CNN
 F 1 "270R" V 5384 2900 50  0001 C CNN
-F 2 "" V 5430 2900 50  0001 C CNN
+F 2 "Resistor_THT:R_Axial_DIN0204_L3.6mm_D1.6mm_P7.62mm_Horizontal" V 5430 2900 50  0001 C CNN
 F 3 "~" H 5500 2900 50  0001 C CNN
 	1    5500 2900
@@
 F 0 "R17" V 5500 3000 50  0000 C CNN
 F 1 "270R" V 5384 3000 50  0001 C CNN
-F 2 "" V 5430 3000 50  0001 C CNN
+F 2 "Resistor_THT:R_Axial_DIN0204_L3.6mm_D1.6mm_P7.62mm_Horizontal" V 5430 3000 50  0001 C CNN
 F 3 "~" H 5500 3000 50  0001 C CNN
 	1    5500 3000
@@
 F 0 "R18" V 5500 3100 50  0000 C CNN
 F 1 "270R" V 5384 3100 50  0001 C CNN
-F 2 "" V 5430 3100 50  0001 C CNN
+F 2 "Resistor_THT:R_Axial_DIN0204_L3.6mm_D1.6mm_P7.62mm_Horizontal" V 5430 3100 50  0001 C CNN
 F 3 "~" H 5500 3100 50  0001 C CNN
 	1    5500 3100
@@
 F 0 "R19" V 5500 3200 50  0000 C CNN
 F 1 "270R" V 5384 3200 50  0001 C CNN
-F 2 "" V 5430 3200 50  0001 C CNN
+F 2 "Resistor_THT:R_Axial_DIN0204_L3.6mm_D1.6mm_P7.62mm_Horizontal" V 5430 3200 50  0001 C CNN
 F 3 "~" H 5500 3200 50  0001 C CNN
 	1    5500 3200
@@
 F 0 "R20" V 5500 3300 50  0000 C CNN
 F 1 "270R" V 5384 3300 50  0001 C CNN
-F 2 "" V 5430 3300 50  0001 C CNN
+F 2 "Resistor_THT:R_Axial_DIN0204_L3.6mm_D1.6mm_P7.62mm_Horizontal" V 5430 3300 50  0001 C CNN
 F 3 "~" H 5500 3300 50  0001 C CNN
 	1    5500 3300
@@
 F 0 "R21" V 5500 4450 50  0000 C CNN
 F 1 "270R" V 5384 4450 50  0001 C CNN
-F 2 "" V 5430 4450 50  0001 C CNN
+F 2 "Resistor_THT:R_Axial_DIN0204_L3.6mm_D1.6mm_P7.62mm_Horizontal" V 5430 4450 50  0001 C CNN
 F 3 "~" H 5500 4450 50  0001 C CNN
 	1    5500 4450
@@
 F 0 "R22" V 5500 4550 50  0000 C CNN
 F 1 "270R" V 5384 4550 50  0001 C CNN
-F 2 "" V 5430 4550 50  0001 C CNN
+F 2 "Resistor_THT:R_Axial_DIN0204_L3.6mm_D1.6mm_P7.62mm_Horizontal" V 5430 4550 50  0001 C CNN
 F 3 "~" H 5500 4550 50  0001 C CNN
 	1    5500 4550
@@
 F 0 "R23" V 5500 4650 50  0000 C CNN
 F 1 "270R" V 5384 4650 50  0001 C CNN
-F 2 "" V 5430 4650 50  0001 C CNN
+F 2 "Resistor_THT:R_Axial_DIN0204_L3.6mm_D1.6mm_P7.62mm_Horizontal" V 5430 4650 50  0001 C CNN
 F 3 "~" H 5500 4650 50  0001 C CNN
 	1    5500 4650
@@
 F 0 "R24" V 5500 4750 50  0000 C CNN
 F 1 "270R" V 5384 4750 50  0001 C CNN
-F 2 "" V 5430 4750 50  0001 C CNN
+F 2 "Resistor_THT:R_Axial_DIN0204_L3.6mm_D1.6mm_P7.62mm_Horizontal" V 5430 4750 50  0001 C CNN
 F 3 "~" H 5500 4750 50  0001 C CNN
 	1    5500 4750
@@
 F 0 "R25" V 5500 4850 50  0000 C CNN
 F 1 "270R" V 5384 4850 50  0001 C CNN
-F 2 "" V 5430 4850 50  0001 C CNN
+F 2 "Resistor_THT:R_Axial_DIN0204_L3.6mm_D1.6mm_P7.62mm_Horizontal" V 5430 4850 50  0001 C CNN
 F 3 "~" H 5500 4850 50  0001 C CNN
 	1    5500 4850
@@
 F 0 "R26" V 5500 4950 50  0000 C CNN
 F 1 "270R" V 5384 4950 50  0001 C CNN
-F 2 "" V 5430 4950 50  0001 C CNN
+F 2 "Resistor_THT:R_Axial_DIN0204_L3.6mm_D1.6mm_P7.62mm_Horizontal" V 5430 4950 50  0001 C CNN
 F 3 "~" H 5500 4950 50  0001 C CNN
 	1    5500 4950
@@
 F 0 "R27" V 5500 5050 50  0000 C CNN
 F 1 "270R" V 5384 5050 50  0001 C CNN
-F 2 "" V 5430 5050 50  0001 C CNN
+F 2 "Resistor_THT:R_Axial_DIN0204_L3.6mm_D1.6mm_P7.62mm_Horizontal" V 5430 5050 50  0001 C CNN
 F 3 "~" H 5500 5050 50  0001 C CNN
 	1    5500 5050
@@
 F 0 "R28" V 5550 6200 50  0000 C CNN
 F 1 "270R" V 5434 6200 50  0001 C CNN
-F 2 "" V 5480 6200 50  0001 C CNN
+F 2 "Resistor_THT:R_Axial_DIN0204_L3.6mm_D1.6mm_P7.62mm_Horizontal" V 5480 6200 50  0001 C CNN
 F 3 "~" H 5550 6200 50  0001 C CNN
 	1    5550 6200
@@
 F 0 "R29" V 5550 6300 50  0000 C CNN
 F 1 "270R" V 5434 6300 50  0001 C CNN
-F 2 "" V 5480 6300 50  0001 C CNN
+F 2 "Resistor_THT:R_Axial_DIN0204_L3.6mm_D1.6mm_P7.62mm_Horizontal" V 5480 6300 50  0001 C CNN
 F 3 "~" H 5550 6300 50  0001 C CNN
 	1    5550 6300
@@
 F 0 "R30" V 5550 6400 50  0000 C CNN
 F 1 "270R" V 5434 6400 50  0001 C CNN
-F 2 "" V 5480 6400 50  0001 C CNN
+F 2 "Resistor_THT:R_Axial_DIN0204_L3.6mm_D1.6mm_P7.62mm_Horizontal" V 5480 6400 50  0001 C CNN
 F 3 "~" H 5550 6400 50  0001 C CNN
 	1    5550 6400
@@
 F 0 "R31" V 5550 6500 50  0000 C CNN
 F 1 "270R" V 5434 6500 50  0001 C CNN
-F 2 "" V 5480 6500 50  0001 C CNN
+F 2 "Resistor_THT:R_Axial_DIN0204_L3.6mm_D1.6mm_P7.62mm_Horizontal" V 5480 6500 50  0001 C CNN
 F 3 "~" H 5550 6500 50  0001 C CNN
 	1    5550 6500
@@
 F 0 "R32" V 5550 6600 50  0000 C CNN
 F 1 "270R" V 5434 6600 50  0001 C CNN
-F 2 "" V 5480 6600 50  0001 C CNN
+F 2 "Resistor_THT:R_Axial_DIN0204_L3.6mm_D1.6mm_P7.62mm_Horizontal" V 5480 6600 50  0001 C CNN
 F 3 "~" H 5550 6600 50  0001 C CNN
 	1    5550 6600
@@
 F 0 "R33" V 5550 6700 50  0000 C CNN
 F 1 "270R" V 5434 6700 50  0001 C CNN
-F 2 "" V 5480 6700 50  0001 C CNN
+F 2 "Resistor_THT:R_Axial_DIN0204_L3.6mm_D1.6mm_P7.62mm_Horizontal" V 5480 6700 50  0001 C CNN
 F 3 "~" H 5550 6700 50  0001 C CNN
 	1    5550 6700
@@
 F 0 "R34" V 5550 6800 50  0000 C CNN
 F 1 "270R" V 5434 6800 50  0001 C CNN
-F 2 "" V 5480 6800 50  0001 C CNN
+F 2 "Resistor_THT:R_Axial_DIN0204_L3.6mm_D1.6mm_P7.62mm_Horizontal" V 5480 6800 50  0001 C CNN
 F 3 "~" H 5550 6800 50  0001 C CNN
 	1    5550 6800
@@
 F 0 "R6" V 7150 1000 50  0000 C CNN
 F 1 "270R" V 7034 1000 50  0001 C CNN
-F 2 "" V 7080 1000 50  0001 C CNN
+F 2 "Resistor_THT:R_Axial_DIN0204_L3.6mm_D1.6mm_P7.62mm_Horizontal" V 7080 1000 50  0001 C CNN
 F 3 "~" H 7150 1000 50  0001 C CNN
 	1    7150 1000
