File: 2-provas/trabalhos-substitutos/2020-ete103-p2-n/questao-03-04.sch (KiCad schematic (older format))
At the start: 7 parts

Commit message: Conclusão da elaboração da prova.
Parts:
- added R1: 1kΩ, symbol Device:R_US
- added R2: 2k2Ω, symbol Device:R_US
- added R3: 4k7Ω, symbol Device:R_US
- added V1: 10V, symbol Device:Battery_Cell
- added V2: 5V, symbol Device:Battery_Cell
- added V3: 2,5V, symbol Device:Battery_Cell
- added Vx: seta_tensao_longa, symbol Pessoal:seta_tensao_longa
Connections:
- new net: R1.1, V1.1 (+)
- new net: V1.2 (-), V2.2 (-), V3.2 (-)
- new net: R2.1, V2.1 (+)
- new net: R1.2, R2.2, R3.2
- new net: R3.1, V3.1 (+)
Other:
- note added: "Iα"
- note added: "Iβ"
- moved on the sheet: R1, R2, R3, V1, V2, V3, Vx
