File: 2-provas/trabalhos-substitutos/2020-ete103-p2-n/questao-08.sch (KiCad schematic (older format))
At the start: 15 parts, among them SW1 SW_SPST, SW2 SW_SPST, t0 seta_tempo_dupla, t1 seta_tempo

Commit message: Conclusão da elaboração da prova.
Parts:
- added ic(t) (x2): seta_corrente_canto, symbol Pessoal:seta_corrente_canto
- added vc(t), vc(t)?, vr1(t) (x2), vr2(t): seta_tensao_longa, symbol Pessoal:seta_tensao_longa
Other:
- moved on the sheet: C1, R1, R2, R?, SW1, SW2, V1
