File: 1.3-laboratorio/projetos/ponta-de-prova-logica/ponta-de-prova-logica-simplificada/ponta-de-prova-logica-simplificada.sch (KiCad schematic (older format))
At the start: 20 parts, among them J1 Conn_01x02, J2 PONTA DE PROVA, SW1 SW_DPDT_x2, U1 LM339

Commit message: Diversas referências sobre SMD da Vishay. Construção de início de notas técnicas para projeto de circuito eletrônicos. Lista de materiais agrupados para a Ponta de Prova Lógica e Circuito para Depuração 01.
Parts:
- U1: Observação (none) -> http://www.ti.com/lit/ds/symlink/lm339.pdf
Changed lines of the file:
@@
 F 1 "LM339" H 7700 4350 50  0000 C CNN
 F 2 "Package_DIP:DIP-14_W7.62mm_Socket_LongPads" H 7500 4300 50  0001 C CNN
-F 3 "http://www.ti.com/lit/ds/symlink/lm339.pdf" H 7600 4400 50  0001 C CNN
+F 3 "http://pdf.datasheetcatalog.com/datasheet/nationalsemiconductor/DS005706.PDF" H 7600 4400 50  0001 C CNN
 	1    7550 4200
 	1    0    0    -1
@@
 F 1 "LM339" H 7700 3500 50  0000 C CNN
 F 2 "Package_DIP:DIP-14_W7.62mm_Socket_LongPads" H 7500 3450 50  0001 C CNN
-F 3 "http://www.ti.com/lit/ds/symlink/lm339.pdf" H 7600 3550 50  0001 C CNN
+F 3 "http://pdf.datasheetcatalog.com/datasheet/nationalsemiconductor/DS005706.PDF" H 7600 3550 50  0001 C CNN
 	2    7550 3350
 	1    0    0    -1
@@
 F 1 "LM339" H 3850 4500 50  0000 C CNN
 F 2 "Package_DIP:DIP-14_W7.62mm_Socket_LongPads" H 3650 4450 50  0001 C CNN
-F 3 "http://www.ti.com/lit/ds/symlink/lm339.pdf" H 3750 4550 50  0001 C CNN
+F 3 "http://pdf.datasheetcatalog.com/datasheet/nationalsemiconductor/DS005706.PDF" H 3750 4550 50  0001 C CNN
+F 4 "http://www.ti.com/lit/ds/symlink/lm339.pdf" H 3700 4350 50  0001 C CNN "Observação"
 	3    3700 4350
 	1    0    0    -1
@@
 F 1 "LM339" H 3850 5100 50  0000 C CNN
 F 2 "Package_DIP:DIP-14_W7.62mm_Socket_LongPads" H 3650 5050 50  0001 C CNN
-F 3 "http://www.ti.com/lit/ds/symlink/lm339.pdf" H 3750 5150 50  0001 C CNN
+F 3 "http://pdf.datasheetcatalog.com/datasheet/nationalsemiconductor/DS005706.PDF" H 3750 5150 50  0001 C CNN
 	4    3700 4950
 	1    0    0    -1
@@
 F 1 "LM339" H 7508 3305 50  0001 L CNN
 F 2 "Package_DIP:DIP-14_W7.62mm_Socket_LongPads" H 7500 3450 50  0001 C CNN
-F 3 "http://www.ti.com/lit/ds/symlink/lm339.pdf" H 7600 3550 50  0001 C CNN
+F 3 "http://pdf.datasheetcatalog.com/datasheet/nationalsemiconductor/DS005706.PDF" H 7600 3550 50  0001 C CNN
 	5    7550 3350
 	1    0    0    -1
