File: 1.3-laboratorio/projetos/sinalizador-noturno/sinalizador-noturno.sch (KiCad schematic (older format))
At the start: 14 parts, among them P1 100k, U1 4093

Commit message: Atualização do projeto 'Sinalizador Noturno'. Inclusão do projeto 'Semáforo'.
Parts:
- gave numbers to parts that had none: 1
Connections:
- wire segments 52 -> 58
Changed lines of the file:
@@
 	4850 4750 4950 4750
 Wire Wire Line
-	4950 2550 4950 3000
-Wire Wire Line
-	4950 1800 4950 2250
+	4950 2550 4950 2900
+Wire Wire Line
+	4950 1800 4950 1900
 Wire Wire Line
 	3650 3800 3400 3800
@@
 	3650 5700 3650 5350
 $Comp
-L Transistor_BJT:BC328 Q?
+L Transistor_BJT:BC328 Q1
 U 1 1 617014EC
 P 8150 4650
-F 0 "Q?" H 8341 4604 50  0000 L CNN
+F 0 "Q1" H 8341 4604 50  0000 L CNN
 F 1 "BC328" H 8341 4695 50  0000 L CNN
 F 2 "Package_TO_SOT_THT:TO-92_Inline" H 8350 4575 50  0001 L CIN
@@
 EndData
 $EndBitmap
+$Comp
+L power:PWR_FLAG #FLG0101
+U 1 1 61637578
+P 5100 1800
+F 0 "#FLG0101" H 5100 1875 50  0001 C CNN
+F 1 "PWR_FLAG" H 5100 1973 50  0001 C CNN
+F 2 "" H 5100 1800 50  0001 C CNN
+F 3 "~" H 5100 1800 50  0001 C CNN
+	1    5100 1800
+	1    0    0    -1
+$EndComp
+Wire Wire Line
+	5100 1800 5100 1900
+Wire Wire Line
+	5100 1900 4950 1900
+Connection ~ 4950 1900
+Wire Wire Line
+	4950 1900 4950 2250
+$Comp
+L power:PWR_FLAG #FLG0102
+U 1 1 616393DC
+P 5100 3000
+F 0 "#FLG0102" H 5100 3075 50  0001 C CNN
+F 1 "PWR_FLAG" H 5100 3173 50  0001 C CNN
+F 2 "" H 5100 3000 50  0001 C CNN
+F 3 "~" H 5100 3000 50  0001 C CNN
+	1    5100 3000
+	-1   0    0    1
+$EndComp
+Wire Wire Line
+	5100 3000 5100 2900
+Wire Wire Line
+	5100 2900 4950 2900
+Connection ~ 4950 2900
+Wire Wire Line
+	4950 2900 4950 3000
 $EndSCHEMATC

Commit message: Projeto 'Deslocamento de LEDs Alternativo. Pequenas revisões nos outros dois projetos recém-criados. Fonte CC com novos padrões pré-definidos.
Parts:
- U1: value 4093 -> 4093B
- renumbered R2 to LDR1
Changed lines of the file:
@@
 P 4550 4750
 F 0 "U1" H 4750 5000 50  0000 C CNN
-F 1 "4093" H 4750 4900 50  0000 C CNN
+F 1 "4093B" H 4750 4900 50  0000 C CNN
 F 2 "" H 4550 4750 50  0001 C CNN
 F 3 "https://assets.nexperia.com/documents/data-sheet/HEF4093B.pdf" H 4550 4750 50  0001 C CNN
@@
 P 5550 4550
 F 0 "U1" H 5550 4875 50  0000 C CNN
-F 1 "4093" H 5550 4784 50  0000 C CNN
+F 1 "4093B" H 5550 4784 50  0000 C CNN
 F 2 "" H 5550 4550 50  0001 C CNN
 F 3 "https://assets.nexperia.com/documents/data-sheet/HEF4093B.pdf" H 5550 4550 50  0001 C CNN
@@
 P 7200 4650
 F 0 "U1" H 7200 4975 50  0000 C CNN
-F 1 "4093" H 7200 4884 50  0000 C CNN
+F 1 "4093B" H 7200 4884 50  0000 C CNN
 F 2 "" H 7200 4650 50  0001 C CNN
 F 3 "https://assets.nexperia.com/documents/data-sheet/HEF4093B.pdf" H 7200 4650 50  0001 C CNN
@@
 P 6150 2400
 F 0 "U1" H 6380 2446 50  0000 L CNN
-F 1 "4093" H 6380 2355 50  0000 L CNN
+F 1 "4093B" H 6380 2355 50  0000 L CNN
 F 2 "" H 6150 2400 50  0001 C CNN
 F 3 "https://assets.nexperia.com/documents/data-sheet/HEF4093B.pdf" H 6150 2400 50  0001 C CNN
@@
 	6150 2950 6150 2900
 $Comp
-L Device:R_PHOTO R2
+L Device:R_PHOTO LDR1
 U 1 1 616BDE3F
 P 3650 5200
-F 0 "R2" H 3720 5246 50  0000 L CNN
+F 0 "LDR1" H 3720 5246 50  0000 L CNN
 F 1 "GL5516" H 3720 5155 50  0000 L CNN
 F 2 "" V 3700 4950 50  0001 L CNN
@@
 P 6500 4550
 F 0 "U1" H 6500 4875 50  0000 C CNN
-F 1 "4093" H 6500 4784 50  0000 C CNN
+F 1 "4093B" H 6500 4784 50  0000 C CNN
 F 2 "" H 6500 4550 50  0001 C CNN
 F 3 "https://assets.nexperia.com/documents/data-sheet/HEF4093B.pdf" H 6500 4550 50  0001 C CNN
