File: 2-provas/imagens-fontes/kicad/2021-an-p2/carga-e-descarga-de-capacitor.sch (KiCad schematic (older format))
At the start: 7 parts, among them SW1 SW_DP3T, t1 seta_tempo

Commit message: Datasheets novos. Renomeação de alguns datasheets. Bibliotecas do Kicad personalizadas. Pseudo-carimbos para o Xournal. P2 de ETE103/N de 2021.
Parts:
- V1: value 3V -> 10V
- V2: value 10V -> 3V
Changed lines of the file:
@@
 P 4650 2950
 F 0 "V1" H 4768 3046 50  0000 L CNN
-F 1 "3V" H 4768 2955 50  0000 L CNN
+F 1 "10V" H 4768 2955 50  0000 L CNN
 F 2 "" V 4650 3010 50  0001 C CNN
 F 3 "~" V 4650 3010 50  0001 C CNN
@@
 P 5450 2950
 F 0 "V2" H 5568 3046 50  0000 L CNN
-F 1 "10V" H 5568 2955 50  0000 L CNN
+F 1 "3V" H 5568 2955 50  0000 L CNN
 F 2 "" V 5450 3010 50  0001 C CNN
 F 3 "~" V 5450 3010 50  0001 C CNN
