File: 1.3-laboratorio/projetos/dado-digital/dado-digital-completo/kicad/dd_cmos/DD_CMOS.sch (KiCad schematic (older format))
At the start: 45 parts, among them P1 CONN_01X02, P2 CONN_01X02, P4 CONN_01X02, Q1 BC547, SW1 SW_PUSH, U1 4093, U2 4027, U3 CD4511BE, U4 4518, U5 C-1505SR-BW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

Commit message: Concluída a revisão do  esquema elétrico do Dado Digital Completo. Em elaboração, a lista de materiais.
Parts:
- added D2: Verde, symbol Device:LED_ALT
- added R6: 1k, symbol DD_CMOS-rescue:R
- C1: value 1uF -> 1uF/16V; symbol DD_CMOS-rescue:C -> Device:CP1
- C2: value 10uF -> 10uF/16V; symbol DD_CMOS-rescue:C -> Device:CP1
Connections:
- net labels added: Ctrl
- net labels removed: GNDA, VSS
- wire segments 239 -> 244
Other:
- note added: ""Displays""
- note added: "Atuador"
- note added: "Botão e\n"deboucing""
- note added: "Capacitores de "bypass""
- note added: "Cargas"
- note added: "Comparador"
- note added: "Contadores"
- note added: "Controle da\n Contagem"
- note added: "Decodificadores"
- note added: "Oscilador"
- note added: "POR"
- note added: "Para f ≅ 100Hz:\n\n C = 22 nF\n\n ou\n\n RA = RB = 4k7Ω"
- note removed: "Capacitores de bypass\n"
- note removed: "Para f ≅ 100Hz:\n\n C = 22 nF\n\n ou\n\n RA = RB = 4.7e3"
- moved on the sheet: Q1, U4B
Changed lines of the file:
@@
 Sheet 1 1
 Title "Dado Digital - CMOS"
-Date "Primeiro Semestre/2017"
+Date "2022-02-02"
 Rev "1.0"
 Comp "ETE102 - Fundamentos de Circuitos Digitais"
@@
 $EndComp
 $Comp
-L DD_CMOS-rescue:C C1
+L Device:CP1 C1
 U 1 1 57427337
 P 2200 1950
 F 0 "C1" H 2225 2050 50  0001 L CNN
-F 1 "1uF" H 2225 1850 50  0000 L CNN
+F 1 "1uF/16V" H 2225 1850 50  0000 L CNN
 F 2 "" H 2238 1800 50  0000 C CNN
 F 3 "" H 2200 1950 50  0000 C CNN
@@
 L power:VDD #PWR03
 U 1 1 57427413
-P 3200 850
-F 0 "#PWR03" H 3200 700 50  0001 C CNN
-F 1 "VDD" H 3200 1000 50  0000 C CNN
-F 2 "" H 3200 850 50  0000 C CNN
-F 3 "" H 3200 850 50  0000 C CNN
-	1    3200 850
+P 3450 850
+F 0 "#PWR03" H 3450 700 50  0001 C CNN
+F 1 "VDD" H 3450 1000 50  0000 C CNN
+F 2 "" H 3450 850 50  0000 C CNN
+F 3 "" H 3450 850 50  0000 C CNN
+	1    3450 850
 	1    0    0    -1
 $EndComp
@@
 L power:GND #PWR04
 U 1 1 574277F3
-P 5300 3050
-F 0 "#PWR04" H 5300 2800 50  0001 C CNN
-F 1 "GND" H 5300 2900 50  0000 C CNN
-F 2 "" H 5300 3050 50  0000 C CNN
-F 3 "" H 5300 3050 50  0000 C CNN
-	1    5300 3050
+P 5250 3050
+F 0 "#PWR04" H 5250 2800 50  0001 C CNN
+F 1 "GND" H 5250 2900 50  0000 C CNN
+F 2 "" H 5250 3050 50  0000 C CNN
+F 3 "" H 5250 3050 50  0000 C CNN
+	1    5250 3050
 	1    0    0    -1
 $EndComp
@@
 $EndComp
 $Comp
-L DD_CMOS-rescue:C C2
+L Device:CP1 C2
 U 1 1 57427E77
 P 2200 3650
 F 0 "C2" H 2225 3750 50  0001 L CNN
-F 1 "10uF" H 2225 3550 50  0000 L CNN
+F 1 "10uF/16V" H 2225 3550 50  0000 L CNN
 F 2 "" H 2238 3500 50  0000 C CNN
 F 3 "" H 2200 3650 50  0000 C CNN
@@
 L DD_CMOS-rescue:R R3
 U 1 1 5742C9F0
-P 9350 5550
-F 0 "R3" V 9430 5550 50  0001 C CNN
-F 1 "1k" V 9350 5550 50  0000 C CNN
-F 2 "" V 9280 5550 50  0000 C CNN
-F 3 "" H 9350 5550 50  0000 C CNN
-	1    9350 5550
+P 9350 5650
+F 0 "R3" V 9430 5650 50  0000 C CNN
+F 1 "1k" V 9350 5650 50  0000 C CNN
+F 2 "" V 9280 5650 50  0000 C CNN
+F 3 "" H 9350 5650 50  0000 C CNN
+	1    9350 5650
 	0    -1   -1   0
 $EndComp
@@
 L DD_CMOS-rescue:BC549 Q1
 U 1 1 5742CA8F
-P 9800 5550
-F 0 "Q1" H 10000 5625 50  0000 L CNN
-F 1 "BC547" H 10000 5550 50  0000 L CNN
-F 2 "TO-92" H 10000 5475 50  0001 L CIN
-F 3 "" H 9800 5550 50  0000 L CNN
-	1    9800 5550
+P 9800 5650
+F 0 "Q1" H 10000 5725 50  0000 L CNN
+F 1 "BC547" H 10000 5650 50  0000 L CNN
+F 2 "TO-92" H 10000 5575 50  0001 L CIN
+F 3 "" H 9800 5650 50  0000 L CNN
+	1    9800 5650
 	1    0    0    -1
 $EndComp
@@
 L power:GND #PWR09
 U 1 1 5742CC47
-P 9900 5950
-F 0 "#PWR09" H 9900 5700 50  0001 C CNN
-F 1 "GND" H 9900 5800 50  0000 C CNN
-F 2 "" H 9900 5950 50  0000 C CNN
-F 3 "" H 9900 5950 50  0000 C CNN
-	1    9900 5950
+P 9900 6050
+F 0 "#PWR09" H 9900 5800 50  0001 C CNN
+F 1 "GND" H 9900 5900 50  0000 C CNN
+F 2 "" H 9900 6050 50  0000 C CNN
+F 3 "" H 9900 6050 50  0000 C CNN
+	1    9900 6050
 	1    0    0    -1
 $EndComp
@@
 	6350 1350 6900 1350
 Wire Wire Line
-	6350 2550 6750 2550
+	6300 2550 6750 2550
 Wire Wire Line
 	6750 2550 7600 2550
 Wire Wire Line
-	6350 2650 6650 2650
+	6300 2650 6650 2650
 Wire Wire Line
 	6650 2650 7600 2650
 Wire Wire Line
-	6350 2750 6550 2750
+	6300 2750 6550 2750
 Wire Wire Line
 	6550 2750 7600 2750
 Wire Wire Line
-	6350 2850 6450 2850
+	6300 2850 6450 2850
 Wire Wire Line
 	6450 2850 7600 2850
@@
 Connection ~ 6450 2850
 Wire Wire Line
-	9900 5750 9900 5950
+	9900 5850 9900 6050
 Wire Wire Line
 	8600 1050 9300 1050
@@
 	6350 2250 6350 1350
 Wire Wire Line
-	5200 2250 6350 2250
+	5150 2250 6350 2250
 Connection ~ 6350 1350
 Wire Wire Line
@@
 	9900 5250 9900 5300
 Wire Wire Line
-	9900 5300 9900 5350
+	9900 5300 9900 5450
 Wire Wire Line
 	9550 5300 9900 5300
@@
 	9550 4600 9550 4800
 Wire Wire Line
-	5350 2650 5300 2650
-Wire Wire Line
-	5300 2650 5300 3050
+	5300 2650 5250 2650
+Wire Wire Line
+	5250 2650 5250 3050
 Wire Wire Line
 	1750 1550 2200 1550
@@
 	4750 1250 5300 1250
 Wire Wire Line
-	5200 2850 5200 2250
+	5150 2850 5150 2250
 Wire Wire Line
 	4750 3400 4750 2750
@@
 	4750 2750 4750 1250
 Wire Wire Line
-	5350 2750 4750 2750
+	5300 2750 4750 2750
 Connection ~ 4750 2750
 Wire Wire Line
@@
 	3850 3400 4750 3400
 Wire Wire Line
-	5200 2850 5350 2850
+	5150 2850 5300 2850
 Wire Wire Line
 	5200 1350 5300 1350
@@
 $EndComp
 Wire Wire Line
-	9500 5550 9600 5550
+	9500 5650 9600 5650
 Wire Wire Line
 	9550 5300 9550 5100
@@
 	7400 4600 7500 4600
 Wire Wire Line
-	9100 5550 9200 5550
+	9100 5650 9200 5650
 $Comp
 L DD_CMOS-rescue:CONN_01X02 P1
@@
 	1050 1500 1050 1550
 $Comp
-L power:VSS #PWR021
+L power:PWR_FLAG #PWR021
 U 1 1 574FD29A
 P 1250 1050
 F 0 "#PWR021" H 1250 900 50  0001 C CNN
-F 1 "VSS" H 1250 1200 50  0000 C CNN
+F 1 "PWR_FLAG" H 1250 1200 50  0001 C CNN
 F 2 "" H 1250 1050 50  0000 C CNN
 F 3 "" H 1250 1050 50  0000 C CNN
@@
 	1050 1650 1050 1700
 $Comp
-L power:GNDA #PWR026
-U 1 1 574FFFAC
-P 1050 1700
-F 0 "#PWR026" H 1050 1450 50  0001 C CNN
-F 1 "GNDA" H 1050 1550 50  0000 C CNN
-F 2 "" H 1050 1700 50  0000 C CNN
-F 3 "" H 1050 1700 50  0000 C CNN
-	1    1050 1700
-	1    0    0    -1
-$EndComp
-$Comp
 L DD_CMOS-rescue:FINDER-40.51 RL1
 U 1 1 575012BB
@@
 Text Notes 700  1700 1    60   ~ 0
 +12V
-Text Notes 10400 1100 3    60   ~ 0
+Text Notes 9500 850  0    60   ~ 0
 unidade
-Text Notes 10400 2950 1    60   ~ 0
+Text Notes 9850 2350 2    60   ~ 0
 dezena
 Text Notes 11050 5550 1    60   ~ 0
@@
 	2950 1550 3550 1550
 Wire Wire Line
-	3550 1650 3200 1650
-Wire Wire Line
-	3550 1450 3200 1450
-Connection ~ 3200 1450
-Wire Wire Line
-	3200 1450 3200 1650
-Wire Wire Line
-	3200 850  3200 1450
+	3550 1650 3450 1650
+Wire Wire Line
+	3550 1450 3450 1450
+Connection ~ 3450 1450
+Wire Wire Line
+	3450 1450 3450 1650
+Wire Wire Line
+	3450 850  3450 1450
 Wire Wire Line
 	4250 1450 4150 1450
@@
 L 4xxx:4518 U4
 U 2 1 62009603
-P 5850 2650
-F 0 "U4" H 5850 3017 50  0000 C CNN
-F 1 "4518" H 5850 2926 50  0000 C CNN
-F 2 "" H 5850 2650 50  0001 C CNN
-F 3 "http://www.intersil.com/content/dam/Intersil/documents/cd45/cd4518bms-20bms.pdf" H 5850 2650 50  0001 C CNN
-	2    5850 2650
+P 5800 2650
+F 0 "U4" H 5800 3017 50  0000 C CNN
+F 1 "4518" H 5800 2926 50  0000 C CNN
+F 2 "" H 5800 2650 50  0001 C CNN
+F 3 "http://www.intersil.com/content/dam/Intersil/documents/cd45/cd4518bms-20bms.pdf" H 5800 2650 50  0001 C CNN
+	2    5800 2650
 	1    0    0    -1
 $EndComp
@@
 U 1 1 6212A212
 P 10100 1350
-F 0 "U5" H 10100 2017 50  0000 C CNN
-F 1 "C-1505SR-BW" H 10100 1926 50  0000 C CNN
+F 0 "U5" H 10100 1900 50  0000 C CNN
+F 1 "C-1505SR-BW" V 10350 1500 50  0000 C CNN
 F 2 "Display_7Segment:SBC18-11SURKCGKWA" H 9370 640 50  0001 L CNN
 F 3 "https://www.datasheetarchive.com/pdf/download.php?id=95807997a35626b3d5d4ddbe5548a7f1a69f20&type=M&term=A1505S" H 10100 1540 50  0001 L CNN
@@
 U 1 1 6216BF63
 P 10100 2850
-F 0 "U7" H 10100 3517 50  0000 C CNN
-F 1 "C-1505SR-BW" H 10100 3426 50  0000 C CNN
+F 0 "U7" H 10100 3400 50  0000 C CNN
+F 1 "C-1505SR-BW" V 10350 3000 50  0000 C CNN
 F 2 "Display_7Segment:SBC18-11SURKCGKWA" H 9370 2140 50  0001 L CNN
 F 3 "https://www.datasheetarchive.com/pdf/download.php?id=95807997a35626b3d5d4ddbe5548a7f1a69f20&type=M&term=A1505S" H 10100 3040 50  0001 L CNN
@@
 	8700 4500 9100 4500
 Wire Wire Line
-	9100 4500 9100 5550
+	9100 4500 9100 5650
 Wire Wire Line
 	1750 4600 1750 4550
@@
 	1    0    0    -1
 $EndComp
-Text Notes 3950 4500 0    60   ~ 0
-Capacitores de bypass\n
+Text Notes 3925 4500 0    60   ~ 0
+Capacitores de "bypass"
 Text Notes 3900 4750 0    60   ~ 0
 (posicioná-los próximos\n    aos CIs indicados)
@@
 D ≅ 33%
 Text Notes 4850 7500 0    50   ~ 0
-Para f ≅ 100Hz:\n\n  C = 22 nF\n\n  ou\n\n  RA = RB = 4.7e3
+Para f ≅ 100Hz:\n\n  C = 22 nF\n\n  ou\n\n  RA = RB = 4k7Ω
 Wire Notes Line
 	4800 6900 5650 6900
@@
 Text Notes 1900 4500 0    60   ~ 0
 Pinos de alimentação de\n     CIs multiparte
+Text Notes 2500 2950 0    60   ~ 0
+POR
+Text Notes 2400 1100 0    60   ~ 0
+  Botão e\n"deboucing"
+Wire Wire Line
+	7500 4500 7350 4500
+Text Label 7350 4500 0    60   ~ 0
+Ctrl
+Text Label 4650 1800 2    60   ~ 0
+Ctrl
+Wire Wire Line
+	4650 1650 4650 1800
+Connection ~ 4650 1650
+Text Notes 3650 850  0    60   ~ 0
+Controle da\n Contagem
+Text Notes 5550 1900 0    60   ~ 0
+Contadores
+Text Notes 7750 700  0    60   ~ 0
+Decodificadores
+Text Notes 9875 700  0    60   ~ 0
+"Displays"
+Text Notes 7800 6100 0    60   ~ 0
+Comparador
+Text Notes 9950 4250 0    60   ~ 0
+Atuador
+Text Notes 10600 5750 0    60   ~ 0
+Cargas
+Text Notes 3650 6100 0    60   ~ 0
+Oscilador
+$Comp
+L power:Earth #PWR0101
+U 1 1 62047A03
+P 1050 1700
+F 0 "#PWR0101" H 1050 1450 50  0001 C CNN
+F 1 "Earth" H 1050 1550 50  0001 C CNN
+F 2 "" H 1050 1700 50  0001 C CNN
+F 3 "~" H 1050 1700 50  0001 C CNN
+	1    1050 1700
+	1    0    0    -1
+$EndComp
+$Comp
+L DD_CMOS-rescue:R R6
+U 1 1 62049194
+P 10300 5500
+F 0 "R6" H 10370 5546 50  0000 L CNN
+F 1 "1k" H 10370 5455 50  0000 L CNN
+F 2 "" V 10230 5500 50  0000 C CNN
+F 3 "" H 10300 5500 50  0000 C CNN
+	1    10300 5500
+	1    0    0    -1
+$EndComp
+$Comp
+L Device:LED_ALT D2
+U 1 1 6204A61B
+P 10300 5850
+F 0 "D2" V 10339 5732 50  0000 R CNN
+F 1 "Verde" V 10248 5732 50  0000 R CNN
+F 2 "" H 10300 5850 50  0001 C CNN
+F 3 "~" H 10300 5850 50  0001 C CNN
+	1    10300 5850
+	0    -1   -1   0
+$EndComp
+$Comp
+L power:GND #PWR026
+U 1 1 6204AC75
+P 10300 6050
+F 0 "#PWR026" H 10300 5800 50  0001 C CNN
+F 1 "GND" H 10300 5900 50  0000 C CNN
+F 2 "" H 10300 6050 50  0000 C CNN
+F 3 "" H 10300 6050 50  0000 C CNN
+	1    10300 6050
+	1    0    0    -1
+$EndComp
+Wire Wire Line
+	10300 5300 10300 5350
+Wire Wire Line
+	10300 5650 10300 5700
+Wire Wire Line
+	10300 6000 10300 6050
+Connection ~ 10300 5300
 $EndSCHEMATC

Commit message: Pequenas revisões no desenho do esquema elétrico. Conclusão da lista de materiais para compra -- falta conferência final.
Parts:
- removed P1, P2: CONN_01X02, ~, symbol DD_CMOS-rescue:CONN_01X02
- removed P4: CONN_01X02, symbol DD_CMOS-rescue:CONN_01X02
- removed U5, U7: C-1505SR-BW, Display_7Segment:SBC18-11SURKCGKWA, symbol Display_Character:SBC18-11SURKCGKWA
- added J1, J2, J3: Conn_01x02, symbol Connector_Generic:Conn_01x02
- added U5, U7: SM42056-1, Display_7Segment:KCSC02-105, symbol Display_Character:KCSA02-105
Connections:
- net +12V: now also J2.2 (Pin_2)
- net Earth: now also J2.1 (Pin_1), J3.2 (Pin_2)
- net GND: now also J1.1 (Pin_1), U5.3 (CA), U5.8 (CA), U7.3 (CA), U7.8 (CA)
- net VDD: now also J1.2 (Pin_2)
- net at .14.2: now also U5.10 (G)
- net at .13.2: now also U5.9 (F)
- net at .12.2: now also U5.1 (E)
- net at .11.2: now also U5.2 (D)
- net at .10.2: now also U5.4 (C)
- net at .9.2: now also U5.6 (B)
- net at .8.2: now also U5.7 (A)
- net at .7.2: now also U7.10 (G)
- net at .6.2: now also U7.9 (F)
- net at .5.2: now also U7.1 (E)
- net at .4.2: now also U7.2 (D)
- net at .3.2: now also U7.4 (C)
- net at .2.2: now also U7.6 (B)
- net at .1.2: now also U7.7 (A)
- net at R6.1, RL1.11: now also J3.1 (Pin_1)
Other:
- note added: "Para f ≅ 220Hz:\n\n C = 10 nF"
Changed lines of the file:
@@
 Sheet 1 1
 Title "Dado Digital - CMOS"
-Date "2022-02-02"
+Date "2022-02-03"
 Rev "1.0"
 Comp "ETE102 - Fundamentos de Circuitos Digitais"
@@
 Wire Wire Line
 	2200 2300 2200 2100
-$Comp
-L DD_CMOS-rescue:CONN_01X02 P4
-U 1 1 574CE7B0
-P 10800 5350
-F 0 "P4" H 10800 5500 50  0000 C CNN
-F 1 "CONN_01X02" V 10900 5350 50  0001 C CNN
-F 2 "" H 10800 5350 50  0000 C CNN
-F 3 "" H 10800 5350 50  0000 C CNN
-	1    10800 5350
-	1    0    0    -1
-$EndComp
 Wire Wire Line
 	9500 5650 9600 5650
@@
 	9100 5650 9200 5650
 $Comp
-L DD_CMOS-rescue:CONN_01X02 P1
-U 1 1 574F8BD1
-P 800 950
-F 0 "P1" H 800 1100 50  0000 C CNN
-F 1 "CONN_01X02" V 900 950 50  0001 C CNN
-F 2 "~" H 800 950 50  0000 C CNN
-F 3 "" H 800 950 50  0000 C CNN
-	1    800  950
-	-1   0    0    -1
-$EndComp
-$Comp
 L power:GND #PWR016
 U 1 1 574F8DC8
@@
 Wire Wire Line
 	1050 1000 1050 1050
-$Comp
-L DD_CMOS-rescue:CONN_01X02 P2
-U 1 1 574FB283
-P 800 1600
-F 0 "P2" H 800 1750 50  0000 C CNN
-F 1 "CONN_01X02" V 900 1600 50  0001 C CNN
-F 2 "~" H 800 1600 50  0000 C CNN
-F 3 "" H 800 1600 50  0000 C CNN
-	1    800  1600
-	-1   0    0    -1
-$EndComp
 Wire Wire Line
 	1000 1650 1050 1650
@@
 Wire Wire Line
 	7450 3050 7450 3700
-$Comp
-L Display_Character:SBC18-11SURKCGKWA U5
-U 1 1 6212A212
-P 10100 1350
-F 0 "U5" H 10100 1900 50  0000 C CNN
-F 1 "C-1505SR-BW" V 10350 1500 50  0000 C CNN
-F 2 "Display_7Segment:SBC18-11SURKCGKWA" H 9370 640 50  0001 L CNN
-F 3 "https://www.datasheetarchive.com/pdf/download.php?id=95807997a35626b3d5d4ddbe5548a7f1a69f20&type=M&term=A1505S" H 10100 1540 50  0001 L CNN
-	1    10100 1350
-	1    0    0    -1
-$EndComp
 Wire Wire Line
 	9600 1050 9800 1050
@@
 Wire Wire Line
 	9700 1750 9800 1750
-$Comp
-L Display_Character:SBC18-11SURKCGKWA U7
-U 1 1 6216BF63
-P 10100 2850
-F 0 "U7" H 10100 3400 50  0000 C CNN
-F 1 "C-1505SR-BW" V 10350 3000 50  0000 C CNN
-F 2 "Display_7Segment:SBC18-11SURKCGKWA" H 9370 2140 50  0001 L CNN
-F 3 "https://www.datasheetarchive.com/pdf/download.php?id=95807997a35626b3d5d4ddbe5548a7f1a69f20&type=M&term=A1505S" H 10100 3040 50  0001 L CNN
-	1    10100 2850
-	1    0    0    -1
-$EndComp
 Wire Wire Line
 	9600 2550 9800 2550
@@
 Text GLabel 4500 6650 2    60   Input ~ 0
 ck
-Text Notes 4800 6600 0    60   ~ 0
+Text Notes 4850 6450 0    60   ~ 0
 f ≅ 2 Hz
-Text Notes 4800 6750 0    60   ~ 0
+Text Notes 4850 6600 0    60   ~ 0
 D ≅ 33%
-Text Notes 4850 7500 0    50   ~ 0
+Text Notes 4900 7300 0    50   ~ 0
 Para f ≅ 100Hz:\n\n  C = 22 nF\n\n  ou\n\n  RA = RB = 4k7Ω
 Wire Notes Line
-	4800 6900 5650 6900
+	4850 6700 5700 6700
 Wire Notes Line
-	5650 6900 5650 7550
-Wire Notes Line
-	5650 7550 4800 7550
-Wire Notes Line
-	4800 7550 4800 6900
+	5700 7350 4850 7350
 Text Notes 1900 4500 0    60   ~ 0
 Pinos de alimentação de\n     CIs multiparte
@@
 	10300 6000 10300 6050
 Connection ~ 10300 5300
+Text Notes 4900 7650 0    50   ~ 0
+Para f ≅ 220Hz:\n\n  C = 10 nF
+Wire Notes Line
+	5700 7700 4850 7700
+Wire Notes Line
+	5700 6700 5700 7700
+Wire Notes Line
+	4850 6700 4850 7700
+$Comp
+L Connector_Generic:Conn_01x02 J1
+U 1 1 620818EA
+P 800 1000
+F 0 "J1" H 800 800 50  0000 C CNN
+F 1 "Conn_01x02" H 718 766 50  0001 C CNN
+F 2 "" H 800 1000 50  0001 C CNN
+F 3 "~" H 800 1000 50  0001 C CNN
+	1    800  1000
+	-1   0    0    1
+$EndComp
+$Comp
+L Connector_Generic:Conn_01x02 J2
+U 1 1 620839E4
+P 800 1650
+F 0 "J2" H 800 1450 50  0000 C CNN
+F 1 "Conn_01x02" H 718 1416 50  0001 C CNN
+F 2 "" H 800 1650 50  0001 C CNN
+F 3 "~" H 800 1650 50  0001 C CNN
+	1    800  1650
+	-1   0    0    1
+$EndComp
+$Comp
+L Connector_Generic:Conn_01x02 J3
+U 1 1 62084076
+P 10800 5300
+F 0 "J3" H 10750 5400 50  0000 L CNN
+F 1 "Conn_01x02" H 10718 5066 50  0001 C CNN
+F 2 "" H 10800 5300 50  0001 C CNN
+F 3 "~" H 10800 5300 50  0001 C CNN
+	1    10800 5300
+	1    0    0    -1
+$EndComp
+$Comp
+L Display_Character:KCSA02-105 U5
+U 1 1 620A9A20
+P 10100 1350
+F 0 "U5" H 10100 1900 50  0000 C CNN
+F 1 "SM42056-1" V 10350 1450 50  0000 C CNN
+F 2 "Display_7Segment:KCSC02-105" H 10100 750 50  0001 C CNN
+F 3 "http://www.kingbright.com/attachments/file/psearch/000/00/00/KCSA02-105(Ver.10A).pdf" H 9600 1825 50  0001 L CNN
+	1    10100 1350
+	1    0    0    -1
+$EndComp
+$Comp
+L Display_Character:KCSA02-105 U7
+U 1 1 620AA4E5
+P 10100 2850
+F 0 "U7" H 10100 3400 50  0000 C CNN
+F 1 "SM42056-1" V 10350 2950 50  0000 C CNN
+F 2 "Display_7Segment:KCSC02-105" H 10100 2250 50  0001 C CNN
+F 3 "http://www.kingbright.com/attachments/file/psearch/000/00/00/KCSA02-105(Ver.10A).pdf" H 9600 3325 50  0001 L CNN
+	1    10100 2850
+	1    0    0    -1
+$EndComp
 $EndSCHEMATC

Commit message: Pequenos ajustes no esquema elétrico. Esboço da placa do bloco atuador. Complementação da lista de materiais.
Parts:
- removed .1, .10, .11, .12, .13, .14, .2, .3, .4, .5, .6, .7, .9: 220R, symbol DD_CMOS-rescue:R
- added J3, J4: Conn_01x01, Connector_PinHeader_1.00mm:PinHeader_1x01_P1.00mm_Vertical, symbol Connector_Generic:Conn_01x01
- added R10, R11, R12, R13, R14, R15, R16, R17, R18, R19, R7, R8, R9: 220R, Resistor_THT:R_Axial_DIN0207_L6.3mm_D2.5mm_P10.16mm_Horizontal, symbol DD_CMOS-rescue:R
- C1, C2: footprint (none) -> Capacitor_THT:CP_Radial_D5.0mm_P2.50mm
- C10: renamed from C8; footprint (none) -> Capacitor_THT:C_Disc_D5.0mm_W2.5mm_P2.50mm
- C3: renamed from C9; footprint (none) -> Capacitor_THT:CP_Radial_D5.0mm_P2.50mm
- C4: renamed from C3; footprint (none) -> Capacitor_THT:C_Disc_D5.0mm_W2.5mm_P2.50mm
- C5: renamed from C4; footprint (none) -> Capacitor_THT:C_Disc_D5.0mm_W2.5mm_P2.50mm
- C6: renamed from C5; footprint (none) -> Capacitor_THT:C_Disc_D5.0mm_W2.5mm_P2.50mm
- C7: renamed from C10; footprint (none) -> Capacitor_THT:C_Disc_D5.0mm_W2.5mm_P2.50mm
- C8: renamed from C6; footprint (none) -> Capacitor_THT:C_Disc_D5.0mm_W2.5mm_P2.50mm
- C9: renamed from C7; footprint (none) -> Capacitor_THT:C_Disc_D5.0mm_W2.5mm_P2.50mm
- D1: footprint (none) -> Diode_THT:D_DO-34_SOD68_P7.62mm_Horizontal
- D2: footprint (none) -> LED_THT:LED_D3.0mm
- J1, J2: footprint (none) -> TerminalBlock_Phoenix:TerminalBlock_Phoenix_MKDS-1,5-2_1x02_P5.00mm_Horizontal
- J5: renamed from J3; footprint (none) -> TerminalBlock_Phoenix:TerminalBlock_Phoenix_MKDS-1,5-2_1x02_P5.00mm_Horizontal
- Q1: footprint TO-92 -> Package_TO_SOT_THT:TO-92
- R1, R2: footprint (none) -> Resistor_THT:R_Axial_DIN0207_L6.3mm_D2.5mm_P10.16mm_Horizontal
- R20: renamed from R6; footprint (none) -> Resistor_THT:R_Axial_DIN0207_L6.3mm_D2.5mm_P10.16mm_Horizontal
- R3: renamed from R4; footprint (none) -> Resistor_THT:R_Axial_DIN0207_L6.3mm_D2.5mm_P10.16mm_Horizontal
- R4: renamed from R5; footprint (none) -> Resistor_THT:R_Axial_DIN0207_L6.3mm_D2.5mm_P10.16mm_Horizontal
- R5: renamed from R3; footprint (none) -> Resistor_THT:R_Axial_DIN0207_L6.3mm_D2.5mm_P10.16mm_Horizontal
- R6: renamed from .8; footprint (none) -> Resistor_THT:R_Axial_DIN0207_L6.3mm_D2.5mm_P10.16mm_Horizontal
- RL1: footprint (none) -> Relay_THT:Relay_SPDT_SANYOU_SRD_Series_Form_C
- SW1: footprint (none) -> Button_Switch_THT:SW_PUSH_6mm
- U1: footprint (none) -> Package_DIP:DIP-14_W7.62mm_LongPads
- U2: footprint (none) -> Package_DIP:DIP-16_W7.62mm_LongPads
- U3: renamed from U4; footprint (none) -> Package_DIP:DIP-16_W7.62mm_LongPads
- U5: renamed from U8; footprint Texas_Instruments-CD4585B-* -> Package_DIP:DIP-16_W7.62mm_LongPads
- U6: renamed from U3; footprint Texas_Instruments-CD4511BE-* -> Package_DIP:DIP-16_W7.62mm_LongPads
- U7: renamed from U6; footprint Texas_Instruments-CD4511BE-* -> Package_DIP:DIP-16_W7.62mm_LongPads
- U8: renamed from U5; footprint Display_7Segment:KCSC02-105 -> Display_7Segment:7SegmentLED_LTS6760_LTS6780
- U9: renamed from U7; footprint Display_7Segment:KCSC02-105 -> Display_7Segment:7SegmentLED_LTS6760_LTS6780
- renumbered U9 to U4
Connections:
- net Earth: now also D2.1 (K)
- net GND: no longer D2.1 (K)
- net at R5.1: now also J4.1 (Pin_1); no longer U5.3 ((A=B)OUT)
- net at U6.14 (g): now also R12.1
- net at U8.10 (G): now also R12.2
- net at U6.15 (f): now also R11.1
- net at U8.9 (F): now also R11.2
- net at U6.9 (e): now also R10.1
- net at U8.1 (E): now also R10.2
- net at U6.10 (d): now also R9.1
- net at U8.2 (D): now also R9.2
- net at U6.11 (c): now also R8.1
- net at U8.4 (C): now also R8.2
- net at U6.12 (b): now also R7.1
- net at U8.6 (B): now also R7.2
- net at U7.14 (g): now also R19.1
- net at U9.10 (G): now also R19.2
- net at U7.15 (f): now also R18.1
- net at U9.9 (F): now also R18.2
- net at U7.9 (e): now also R17.1
- net at U9.1 (E): now also R17.2
- net at U7.10 (d): now also R16.1
- net at U9.2 (D): now also R16.2
- net at U7.11 (c): now also R15.1
- net at U9.4 (C): now also R15.2
- net at U7.12 (b): now also R14.1
- net at U9.6 (B): now also R14.2
- net at U7.13 (a): now also R13.1
- net at U9.7 (A): now also R13.2
- new net: J3.1 (Pin_1), U5.3 ((A=B)OUT)
Other:
- moved on the sheet: C3, C7, R3, R4, U4
