File: 1.3-laboratorio/projetos/sensor-e-atuador-com-ajuste-digital-de-set-point/simulacoes/sendor-e-atuador-com-ajuste-digital-de-setpoint.sch (KiCad schematic (older format))
At the start: 18 parts, among them U1 OPAMP

Commit message: Simulações para o projeto sendor-e-atuador-com-ajuste-digital-de-setpoint. Esquemas com resolução de exercícios sobre dimensionamento de resistor para LED.
Parts:
- removed R10: 500, symbol pspice:R
- removed R9: 2k, symbol pspice:R
- V1, V2: Spice_Model dc 5 -> dc Vf
- V3: Spice_Model pulse(0 5 50m 500u 500u 50m 100m) -> pulse(0 Vf 50m ts td 50m 100m)
- V4: Spice_Model pulse(0 5 25m 500u 500u 25m 50m) -> pulse(0 Vf 25m ts td 25m 50m)
- V5: Spice_Model pulse(0 5 12.5m 500u 500u 12m 25m) -> pulse(0 Vf 12.5m ts td 12.5m 25m)
- V6: Spice_Model pulse(0 5 6.25m 500u 500u 5.75m 12.5m) -> pulse(0 Vf 6.25m ts td 6.25m 12.5m)
Connections:
- net Vs: now also U1.2 (-)
Other:
- note added: ".param Vf=12\n.param ts = 5us\n.param td = 'ts'"
Changed lines of the file:
@@
 F 3 "~" H 1300 3950 50  0001 C CNN
 F 4 "V" H 1300 3950 50  0001 C CNN "Spice_Primitive"
-F 5 "pulse(0 5 50m 500u 500u 50m 100m)" H 1300 3950 50  0001 C CNN "Spice_Model"
+F 5 "pulse(0 Vf 50m ts td 50m 100m)" H 1300 3950 50  0001 C CNN "Spice_Model"
 F 6 "Y" H 1300 3950 50  0001 C CNN "Spice_Netlist_Enabled"
 	1    1300 3950
@@
 	1500 650  1500 750
 Wire Wire Line
-	6200 2050 6200 2100
-Wire Wire Line
-	6300 2050 6200 2050
-$Comp
-L power:Earth #PWR08
-U 1 1 6325C62A
-P 6200 2100
-F 0 "#PWR08" H 6200 1850 50  0001 C CNN
-F 1 "Earth" H 6200 1950 50  0001 C CNN
-F 2 "" H 6200 2100 50  0001 C CNN
-F 3 "~" H 6200 2100 50  0001 C CNN
-	1    6200 2100
-	1    0    0    -1
-$EndComp
-$Comp
-L pspice:R R9
-U 1 1 6325ABEA
-P 6550 2050
-F 0 "R9" V 6255 2050 50  0000 C CNN
-F 1 "2k" V 6346 2050 50  0000 C CNN
-F 2 "" H 6550 2050 50  0001 C CNN
-F 3 "~" H 6550 2050 50  0001 C CNN
-F 4 "R" H 6550 2050 50  0001 C CNN "Spice_Primitive"
-F 5 "100k" V 6437 2050 50  0000 C CNN "Spice_Model"
-F 6 "Y" H 6550 2050 50  0001 C CNN "Spice_Netlist_Enabled"
-	1    6550 2050
-	0    1    1    0
-$EndComp
-Wire Wire Line
 	6900 1550 7000 1550
 Wire Wire Line
-	6800 2050 6900 2050
-Wire Wire Line
-	6950 2050 6900 2050
-Connection ~ 6900 2050
-Wire Wire Line
 	6900 2050 6900 1550
-Wire Wire Line
-	7700 2050 7450 2050
 Wire Wire Line
 	7700 1450 7700 2050
@@
 Wire Wire Line
 	7600 1450 7700 1450
-$Comp
-L pspice:R R10
-U 1 1 63259F67
-P 7200 2050
-F 0 "R10" V 7313 2050 50  0000 C CNN
-F 1 "500" V 7404 2050 50  0000 C CNN
-F 2 "" H 7200 2050 50  0001 C CNN
-F 3 "~" H 7200 2050 50  0001 C CNN
-F 4 "R" H 7200 2050 50  0001 C CNN "Spice_Primitive"
-F 5 "25k" V 7495 2050 50  0000 C CNN "Spice_Model"
-F 6 "Y" H 7200 2050 50  0001 C CNN "Spice_Netlist_Enabled"
-	1    7200 2050
-	0    1    1    0
-$EndComp
 Wire Wire Line
 	1300 4250 1300 4450
@@
 F 3 "~" H 1300 1550 50  0001 C CNN
 F 4 "V" H 1300 1550 50  0001 C CNN "Spice_Primitive"
-F 5 "dc 5" H 1300 1550 50  0001 C CNN "Spice_Model"
+F 5 "dc Vf" H 1300 1550 50  0001 C CNN "Spice_Model"
 F 6 "Y" H 1300 1550 50  0001 C CNN "Spice_Netlist_Enabled"
 	1    1300 1550
@@
 F 3 "~" H 1300 2600 50  0001 C CNN
 F 4 "V" H 1300 2600 50  0001 C CNN "Spice_Primitive"
-F 5 "dc 5" H 1300 2600 50  0001 C CNN "Spice_Model"
+F 5 "dc Vf" H 1300 2600 50  0001 C CNN "Spice_Model"
 F 6 "Y" H 1300 2600 50  0001 C CNN "Spice_Netlist_Enabled"
 	1    1300 2600
@@
 F 3 "~" H 2250 3950 50  0001 C CNN
 F 4 "V" H 2250 3950 50  0001 C CNN "Spice_Primitive"
-F 5 "pulse(0 5 25m 500u 500u 25m 50m)" H 2250 3950 50  0001 C CNN "Spice_Model"
+F 5 "pulse(0 Vf 25m ts td 25m 50m)" H 2250 3950 50  0001 C CNN "Spice_Model"
 F 6 "Y" H 2250 3950 50  0001 C CNN "Spice_Netlist_Enabled"
 	1    2250 3950
@@
 F 3 "~" H 3200 3950 50  0001 C CNN
 F 4 "V" H 3200 3950 50  0001 C CNN "Spice_Primitive"
-F 5 "pulse(0 5 12.5m 500u 500u 12m 25m)" H 3200 3950 50  0001 C CNN "Spice_Model"
+F 5 "pulse(0 Vf 12.5m ts td 12.5m 25m)" H 3200 3950 50  0001 C CNN "Spice_Model"
 F 6 "Y" H 3200 3950 50  0001 C CNN "Spice_Netlist_Enabled"
 	1    3200 3950
@@
 F 3 "~" H 4150 3950 50  0001 C CNN
 F 4 "V" H 4150 3950 50  0001 C CNN "Spice_Primitive"
-F 5 "pulse(0 5 6.25m 500u 500u 5.75m 12.5m)" H 4150 3950 50  0001 C CNN "Spice_Model"
+F 5 "pulse(0 Vf 6.25m ts td 6.25m 12.5m)" H 4150 3950 50  0001 C CNN "Spice_Model"
 F 6 "Y" H 4150 3950 50  0001 C CNN "Spice_Netlist_Enabled"
 	1    4150 3950
@@
 Text Label 5800 1350 0    50   ~ 0
 Vr2r
+Text Notes 1000 4900 0    50   ~ 0
+.param Vf=12\n.param ts = 5us\n.param td = 'ts'
+Wire Wire Line
+	6900 2050 7700 2050
 $EndSCHEMATC
