File: 1.3-laboratorio/projetos/sensor-e-atuador-com-ajuste-digital-de-set-point/simulacoes/resistor-controlado-por-tensao.kicad_sch (KiCad schematic)
At the start: 4 parts, among them Q1 Q_Dual_NPN_C2C1E1E2

Commit message: Estudos e simulações concluídas para o modelo mais didático do Sensor e Atuador com Ajuste Digital de Set-point. Alguns datasheets adicionados. Modelo docx para provas adicionado.
Parts:
- added R1: R, symbol Device:R
- added R3: 1k, symbol Device:R
- added V3: 0, symbol Device:Battery_Cell
- Q1: Spice_Lib_File vres.lib -> (none); Spice_Model VC_RES1_10K -> (none); Spice_Netlist_Enabled Y -> (none); Spice_Node_Sequence 3 2 1 4 -> (none); Spice_Primitive X -> (none)
- R2: Spice_Model 10k -> (none); Spice_Netlist_Enabled Y -> (none); Spice_Primitive R -> (none)
- V1: value Battery_Cell -> 12; Spice_Model dc 12 -> (none); Spice_Netlist_Enabled Y -> (none); Spice_Primitive V -> (none)
- V2: value Battery_Cell -> 0.5; Spice_Model dc 0.5 -> (none); Spice_Netlist_Enabled Y -> (none); Spice_Primitive V -> (none)
Connections:
- net 0: now also R3.1
- net VCC: now also R1.2
- net Vs: now also V3.2 (-); no longer R2.1
- net Vctrl: now reaches Q1.1 (C2), V2.1 (+)
- new net: R2.1, V3.1 (+)
- new net Vs2: R1.1, R3.2
Other:
- moved on the sheet: R2
