File: 1.3-laboratorio/projetos/sensor-e-atuador-com-ajuste-digital-de-set-point/simulacoes/mais-didatico/sensor-e-atuador-com-ajuste-digital-de-setpoint-sem-vres-mais-didatico.kicad_sch (KiCad schematic)
At the start: 30 parts, among them U1 OPAMP, U2 OPAMP, U3 OPAMP

Commit message: Obtenção dos gráficos Vs x Rldr. Faltam os com a histerese.
Connections:
- net Vu3+ renamed Vcomp
Changed lines of the file:
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@@
     (effects (font (size 1.27 1.27)) (justify left bottom))
   )
-  (label "Vu3+" (at 246.38 133.985 0) (fields_autoplaced)
-    (effects (font (size 1.27 1.27)) (justify left bottom))
+  (label "Vcomp" (at 246.38 144.145 180) (fields_autoplaced)
+    (effects (font (size 1.27 1.27)) (justify right bottom))
   )
   (label "Vsensor" (at 118.11 152.4 0) (fields_autoplaced)
